File: component_tester.sch (KiCad schematic (older format))
At the start: 1 part

Commit message: Work on schematic
Parts:
- removed U?: ATMEGA328-MU, MLF/QFN32, symbol ATMEGA328-MU
- added C1: 1nF, KiCad/Capacitors_SMD.pretty:C_0201, symbol component_tester-eagle-import:C2.5_2
- added C2: 10nF, KiCad/Capacitors_SMD.pretty:C_0201, symbol component_tester-eagle-import:C2,5-3
- added C3: 100nF, KiCad/Capacitors_SMD.pretty:C_0201, symbol component_tester-eagle-import:C5_3
- added C7, C8: 2.2µF, KiCad/Capacitors_SMD.pretty:C_0603, symbol Device:C
- added D1, D3: SB130, component_tester:DIODE-3-5A-V, symbol component_tester-eagle-import:SCHOTTKY-DIODE_RAD3-5-A
- added D2: 1N4001, component_tester:DIODE-3-5A-V, symbol component_tester-eagle-import:DIODE_RAD3-5-A
- added JP1: Battery 9V, component_tester:PINHD-1X02, symbol component_tester-eagle-import:PINHD-1X2-PCB
- added JP2: 7-12V DC, component_tester:PINHD-1X02, symbol component_tester-eagle-import:PINHD-1X2-PCB
- added JP3: ISP, component_tester:ML6, symbol component_tester-eagle-import:ML6
- added JP4: Test-Pins, component_tester:PINHD-1X03, symbol component_tester-eagle-import:PINHD-1X3-PCB
- added JP5: Start Pushbutton, component_tester:PINHD-1X02, symbol component_tester-eagle-import:PINHD-1X2-PCB
- added JP6: Power LED, component_tester:PINHD-1X02, symbol component_tester-eagle-import:PINHD-1X2-PCB
- added L1: 10µH, component_tester:0204_7, symbol component_tester-eagle-import:L-EU0204_7
- added Q1, Q2: BC547, component_tester:TO92, symbol component_tester-eagle-import:BC547
- added Q7: BC328, component_tester:TO92-EBC, symbol component_tester-eagle-import:BC328
- added R1, R3, R5: 680, component_tester:0207_10, symbol component_tester-eagle-import:R-EU_0207_10
- added R10: 33k, component_tester:0207_2V, symbol component_tester-eagle-import:R-EU_0207_2V
- added R11: 10k, component_tester:0207_2V, symbol component_tester-eagle-import:R-EU_0207_2V
- added R12: 3k3, component_tester:0207_2V, symbol component_tester-eagle-import:R-EU_0207_2V
- added R13: 10k, component_tester:0207_10, symbol component_tester-eagle-import:R-EU_0207_10
- added R17, R8: 27k, component_tester:0207_2V, symbol component_tester-eagle-import:R-EU_0207_2V
- added R2, R4, R6: 470k, component_tester:0207_10, symbol component_tester-eagle-import:R-EU_0207_10
- added R7: 3k3, component_tester:0207_10, symbol component_tester-eagle-import:R-EU_0207_10
- added R9: 100k, component_tester:0207_2V, symbol component_tester-eagle-import:R-EU_0207_2V
- added U1: ATmega8/88/168, component_tester:DIL28-3, symbol component_tester-eagle-import:MEGA8-P
- added U2: MCP1702-5002, component_tester:TO92-LOWDROP, symbol component_tester-eagle-import:MCP1702-5002
- added U3: ATmega328P-MMH, Package_DFN_QFN:QFN-28-1EP_4x4mm_P0.45mm_EP2.25x2.25mm, symbol MCU_Microchip_ATmega:ATmega328P-MMH
Connections:
- net labels added: +12V, +5V, +9V, GND, LED_EXT, PB0, PB1, PB2, PB3, PB4, PB5, PC0, PC1, PC2, PC5, PC6, PD6, PD7
- wire segments 0 -> 144
Other:
- note added: "+"
- note added: "-"
- note added: "1"
- note added: "2"
- note added: "3"

Commit message: Schema schemaaa
Parts:
- removed C2: 10nF, KiCad/Capacitors_SMD.pretty:C_0201, symbol component_tester-eagle-import:C2,5-3
- removed C7, C8: 2.2µF, KiCad/Capacitors_SMD.pretty:C_0603, symbol Device:C
- removed D1, D3: SB130, component_tester:DIODE-3-5A-V, symbol component_tester-eagle-import:SCHOTTKY-DIODE_RAD3-5-A
- removed D2: 1N4001, component_tester:DIODE-3-5A-V, symbol component_tester-eagle-import:DIODE_RAD3-5-A
- removed JP1: Battery 9V, component_tester:PINHD-1X02, symbol component_tester-eagle-import:PINHD-1X2-PCB
- removed JP2: 7-12V DC, component_tester:PINHD-1X02, symbol component_tester-eagle-import:PINHD-1X2-PCB
- removed JP6: Power LED, component_tester:PINHD-1X02, symbol component_tester-eagle-import:PINHD-1X2-PCB
- removed L1: 10µH, component_tester:0204_7, symbol component_tester-eagle-import:L-EU0204_7
- removed Q1, Q2: BC547, component_tester:TO92, symbol component_tester-eagle-import:BC547
- removed Q7: BC328, component_tester:TO92-EBC, symbol component_tester-eagle-import:BC328
- removed R10: 33k, component_tester:0207_2V, symbol component_tester-eagle-import:R-EU_0207_2V
- removed R7: 3k3, component_tester:0207_10, symbol component_tester-eagle-import:R-EU_0207_10
- removed R8: 27k, component_tester:0207_2V, symbol component_tester-eagle-import:R-EU_0207_2V
- removed R9: 100k, component_tester:0207_2V, symbol component_tester-eagle-import:R-EU_0207_2V
- removed U1: ATmega8/88/168, component_tester:DIL28-3, symbol component_tester-eagle-import:MEGA8-P
- removed U2: MCP1702-5002, component_tester:TO92-LOWDROP, symbol component_tester-eagle-import:MCP1702-5002
- added J1: USB_B_Micro, digikey/digikey-kicad-library/digikey-footprints.pretty:USB_Micro_B_Female_10118192, symbol Connector_Specialized:USB_B_Micro
- JP3: footprint component_tester:ML6 -> apexelectrix/apex-pin-headers.pretty:2x3-PIN-1.27mm
- JP4: footprint component_tester:PINHD-1X03 -> KiCad/kicad-footprints/Connector_PinHeader_2.54mm.pretty:PinHeader_1x03_P2.54mm_Vertical_SMD_Pin1Left
- JP5: footprint component_tester:PINHD-1X02 -> freetronics/freetronics_kicad_library/freetronics_footprints.pretty:SW_PUSHBUTTON_SMD
Connections:
- net labels removed: +12V, LED_EXT, PD6
- wire segments 144 -> 95
Other:
- note removed: "+"
- note removed: "-"
