File: kicad/component_tester_1.sch (KiCad schematic (older format))
At the start: 65 parts, among them IC1 MEGA48/88/168-AU, IC2 MCP1640, Q1 8 MHz, SW1 TASTER-RACON8SMD, T1 BC847, T2 BSS123, T3 PMV65XP, T5 BSS84, X1 MINI-USB, X10 P3, X11 P1, X12 P2, X2 P1, X3 P3, X4 P1, X5 P2, X6 ISP, X7 P2, X8 P3, X9 STIFTLEISTE_2,54MM_1X3_WI-SMD

Commit message: Delete eagle schematic blocks
Other:
- note removed: ">REV"
- note removed: "Bauteiltester"
Changed lines of the file:
@@
-$EndComp
-$Comp
-L component_tester-eagle-import:DINA4_L #FRAME1
-U 2 0 80664ACC4FD11FDE
-P 7300 8100
-AR Path="/80664ACC4FD11FDE" Ref="#FRAME1"  Part="2"
-AR Path="/5B1C6B30/80664ACC4FD11FDE" Ref="#FRAME1"  Part="2"
-F 0 "#FRAME1" H 7300 8100 50  0001 C CNN
-F 1 "FiFi" H 7300 8100 50  0001 C CNN
-F 2 "" H 7300 8100 50  0001 C CNN
-F 3 "" H 7300 8100 50  0001 C CNN
-	2    7300 8100
-	1    0    0    -1
 $EndComp
 $Comp
@@
 	1    0    0    -1
 $EndComp
-Text Notes 10900 7800 0    100  ~ 0
->REV
-Text Notes 7500 7100 0    254  ~ 0
-Bauteiltester
 Text Notes 2500 7600 0    59   ~ 0
 Knopfzelle

Commit message: Fix some schematic eagle import oddities
Parts:
- removed LCD1: LCD-FFC10-16X2, component_tester:FFC_14P_1MM_TOP, symbol component_tester-eagle-import:LCD-FFC10-16X2TOP
- removed R15: 10k, component_tester:POTI_ACP6-SMD, symbol component_tester-eagle-import:POTI_ACP6SMD
- X1: value MINI-USB -> MICRO-USB
Connections:
- wire segments 236 -> 211
Changed lines of the file:
@@
 $EndDescr
-Wire Wire Line
-	10200 3700 5400 3700
-Wire Wire Line
-	5400 3800 10200 3800
-Wire Wire Line
-	5400 3900 10200 3900
-Wire Wire Line
-	5400 4000 10200 4000
-Wire Wire Line
-	5400 4200 9700 4200
-Wire Wire Line
-	9700 4200 9700 3200
-Wire Wire Line
-	9700 3200 10200 3200
-Wire Wire Line
-	10200 3600 9950 3600
-Wire Wire Line
-	9950 3600 9950 3500
-Wire Wire Line
-	9950 3500 9950 3400
-Wire Wire Line
-	9950 3400 9950 3300
-Wire Wire Line
-	9950 3300 9800 3300
-Wire Wire Line
-	9800 3300 9800 3400
-Wire Wire Line
-	10200 3300 9950 3300
-Wire Wire Line
-	10200 3400 9950 3400
-Wire Wire Line
-	10200 3500 9950 3500
-Connection ~ 9950 3300
-Connection ~ 9950 3400
-Connection ~ 9950 3500
-Text GLabel 10200 3600 0    10   BiDi ~ 0
-GND
 Wire Wire Line
 	1800 3200 1900 3200
@@
 GND
 Wire Wire Line
-	10100 2700 10200 2700
-Text GLabel 10100 2700 0    10   BiDi ~ 0
-GND
-Wire Wire Line
-	10100 3100 10200 3100
-Text GLabel 10100 3100 0    10   BiDi ~ 0
-GND
-Wire Wire Line
 	7100 6800 7100 7200
 Text GLabel 7100 6800 0    10   BiDi ~ 0
@@
 GND
 Wire Wire Line
-	9400 3200 9400 3100
-Text GLabel 9400 3200 0    10   BiDi ~ 0
-GND
-Wire Wire Line
 	1700 6100 1700 6900
 Wire Wire Line
 	1600 6100 1700 6100
-Text GLabel 1700 6100 0    10   BiDi ~ 0
+Text GLabel 1700 6100 1    10   BiDi ~ 0
 GND
 Wire Wire Line
@@
 +5V
 Wire Wire Line
-	9900 2800 10200 2800
-Text Label 9900 2800 0    10   ~ 0
-+5V
-Wire Wire Line
 	5400 1200 5400 1300
 Text Label 5400 1200 0    10   ~ 0
@@
 +5V
 Wire Wire Line
-	9400 2700 9400 2600
-Text Label 9400 2700 0    10   ~ 0
-+5V
-Wire Wire Line
 	2600 2800 2800 2800
 Wire Wire Line
@@
 Connection ~ 5000 7200
 Wire Wire Line
-	10200 3000 9600 3000
-Wire Wire Line
-	9600 3000 9600 4100
-Wire Wire Line
-	9600 4100 5400 4100
-Wire Wire Line
 	5400 3300 5600 3300
 Wire Wire Line
@@
 	5600 1800 5400 1800
 Connection ~ 5400 1800
-Wire Wire Line
-	10200 2900 9600 2900
 Wire Wire Line
 	8100 1400 8100 1700
@@
 Connection ~ 1800 6500
 Connection ~ 1900 6500
-Text GLabel 1600 6500 0    10   BiDi ~ 0
+Text GLabel 1600 6500 1    10   BiDi ~ 0
 VCC
 Wire Wire Line
@@
 Wire Wire Line
 	2000 6400 2000 6000
-Text GLabel 2000 6000 3    70   BiDi ~ 0
+Text GLabel 2000 6000 1    70   BiDi ~ 0
 USBDM
 Wire Wire Line
@@
 Wire Wire Line
 	2200 6300 2200 6000
-Text GLabel 2200 6000 3    70   BiDi ~ 0
+Text GLabel 2200 6000 1    70   BiDi ~ 0
 USBDP
 Wire Wire Line
@@
 Wire Wire Line
 	6600 3100 6600 2200
-Text GLabel 6600 2200 3    70   BiDi ~ 0
+Text GLabel 6600 2200 1    70   BiDi ~ 0
 SEROUT
 Wire Wire Line
@@
 Wire Wire Line
 	2500 6100 2500 6000
-Text GLabel 2500 6000 3    70   BiDi ~ 0
+Text GLabel 2500 6000 1    70   BiDi ~ 0
 SUP_UART
 Wire Wire Line
@@
 AR Path="/5B1C6B30/97C2823C753049C4" Ref="X1"  Part="1"
 F 0 "X1" H 1300 6800 70  0000 L BNN
-F 1 "MINI-USB" H 1300 6700 70  0000 L BNN
+F 1 "MICRO-USB" H 1300 6700 70  0000 L BNN
 F 2 "component_tester:MINI-USB-B5" H 1400 6300 50  0001 C CNN
 F 3 "" H 1400 6300 50  0001 C CNN
@@
 	1    5200 5900
 	1    0    0    -1
-$EndComp
-$Comp
-L component_tester-eagle-import:LCD-FFC10-16X2TOP LCD1
-U 1 0 5F41E3BF808094CA
-P 10600 3400
-AR Path="/5F41E3BF808094CA" Ref="LCD1"  Part="1"
-AR Path="/5B1C6B30/5F41E3BF808094CA" Ref="LCD1"  Part="1"
-F 0 "LCD1" H 9800 3950 59  0000 L BNN
-F 1 "LCD-FFC10-16X2" H 10550 3950 59  0000 L BNN
-F 2 "component_tester:FFC_14P_1MM_TOP" H 10600 3400 50  0001 C CNN
-F 3 "" H 10600 3400 50  0001 C CNN
-	1    10600 3400
-	0    1    1    0
 $EndComp
 $Comp
@@
 $EndComp
 $Comp
-L component_tester-eagle-import:GND #GND3
-U 1 0 21A7002F7679BDCC
-P 9800 3500
-AR Path="/21A7002F7679BDCC" Ref="#GND3"  Part="1"
-AR Path="/5B1C6B30/21A7002F7679BDCC" Ref="#GND03"  Part="1"
-F 0 "#GND03" H 9800 3500 50  0001 C CNN
-F 1 "GND" H 9700 3400 59  0000 L BNN
-F 2 "" H 9800 3500 50  0001 C CNN
-F 3 "" H 9800 3500 50  0001 C CNN
-	1    9800 3500
-	1    0    0    -1
-$EndComp
-$Comp
 L component_tester-eagle-import:R0805 R1
 U 1 0 512AF7C563543E95
@@
 $EndComp
 $Comp
-L component_tester-eagle-import:GND #GND10
-U 1 0 F47101845C69E3
-P 10000 2700
-AR Path="/F47101845C69E3" Ref="#GND10"  Part="1"
-AR Path="/5B1C6B30/F47101845C69E3" Ref="#GND010"  Part="1"
-F 0 "#GND010" H 10000 2700 50  0001 C CNN
-F 1 "GND" H 9900 2600 59  0000 L BNN
-F 2 "" H 10000 2700 50  0001 C CNN
-F 3 "" H 10000 2700 50  0001 C CNN
-	1    10000 2700
-	0    1    1    0
-$EndComp
-$Comp
-L component_tester-eagle-import:+5V #+5V4
-U 1 0 F92D85D269AA9727
-P 9800 2800
-AR Path="/F92D85D269AA9727" Ref="#+5V4"  Part="1"
-AR Path="/5B1C6B30/F92D85D269AA9727" Ref="#+5V04"  Part="1"
-F 0 "#+5V04" H 9800 2800 50  0001 C CNN
-F 1 "+5V" V 9700 2600 59  0000 L BNN
-F 2 "" H 9800 2800 50  0001 C CNN
-F 3 "" H 9800 2800 50  0001 C CNN
-	1    9800 2800
-	0    -1   -1   0
-$EndComp
-$Comp
-L component_tester-eagle-import:GND #GND11
-U 1 0 25F2C17319DA8D48
-P 10000 3100
-AR Path="/25F2C17319DA8D48" Ref="#GND11"  Part="1"
-AR Path="/5B1C6B30/25F2C17319DA8D48" Ref="#GND011"  Part="1"
-F 0 "#GND011" H 10000 3100 50  0001 C CNN
-F 1 "GND" H 9900 3000 59  0000 L BNN
-F 2 "" H 10000 3100 50  0001 C CNN
-F 3 "" H 10000 3100 50  0001 C CNN
-	1    10000 3100
-	0    1    1    0
-$EndComp
-$Comp
 L component_tester-eagle-import:R0805 R10
 U 1 0 B36C6E30D74182C5
@@
 $EndComp
 $Comp
-L component_tester-eagle-import:POTI_ACP6SMD R15
-U 1 0 FBFB61278104E241
-P 9400 2900
-AR Path="/FBFB61278104E241" Ref="R15"  Part="1"
-AR Path="/5B1C6B30/FBFB61278104E241" Ref="R15"  Part="1"
-F 0 "R15" H 9250 3135 59  0001 L BNN
-F 1 "10k" H 9250 3050 59  0001 L BNN
-F 2 "component_tester:POTI_ACP6-SMD" H 9400 2900 50  0001 C CNN
-F 3 "" H 9400 2900 50  0001 C CNN
-	1    9400 2900
-	0    -1   1    0
-$EndComp
-$Comp
-L component_tester-eagle-import:GND #GND15
-U 1 0 CBE454F257B06B4
-P 9400 3300
-AR Path="/CBE454F257B06B4" Ref="#GND15"  Part="1"
-AR Path="/5B1C6B30/CBE454F257B06B4" Ref="#GND015"  Part="1"
-F 0 "#GND015" H 9400 3300 50  0001 C CNN
-F 1 "GND" H 9300 3200 59  0000 L BNN
-F 2 "" H 9400 3300 50  0001 C CNN
-F 3 "" H 9400 3300 50  0001 C CNN
-	1    9400 3300
-	1    0    0    -1
-$EndComp
-$Comp
-L component_tester-eagle-import:+5V #+5V6
-U 1 0 393C5AB363AB7CC1
-P 9400 2500
-AR Path="/393C5AB363AB7CC1" Ref="#+5V6"  Part="1"
-AR Path="/5B1C6B30/393C5AB363AB7CC1" Ref="#+5V06"  Part="1"
-F 0 "#+5V06" H 9400 2500 50  0001 C CNN
-F 1 "+5V" V 9300 2300 59  0000 L BNN
-F 2 "" H 9400 2500 50  0001 C CNN
-F 3 "" H 9400 2500 50  0001 C CNN
-	1    9400 2500
-	1    0    0    -1
-$EndComp
-$Comp
 L component_tester-eagle-import:GND #GND16
 U 1 0 8316678299D4D269
@@
 	1    0    0    -1
 $EndComp
-Text Notes 2500 7600 0    59   ~ 0
+Text Notes 2075 7475 0    59   ~ 0
 Knopfzelle
-Text Notes 2600 7600 0    59   ~ 0
+Text Notes 2100 7575 0    59   ~ 0
 CR2032
 Text Notes 7300 1200 0    85   ~ 0
@@
 Text Notes 9800 1200 0    85   ~ 0
 Reserve
-Text Notes 1100 4300 0    127  ~ 0
+Text Notes 1100 2000 0    127  ~ 0
 K.-H. Kübbeler, DF3DCB, DH8GHH
 Text GLabel 2600 7200 0    10   BiDi ~ 0

Commit message: Switch resistors and caps to 0201 where possible
Parts:
- C1, C2, C3, C6: footprint component_tester:C0805 -> KiCad/Capacitors_SMD.pretty:C_0201
- C10, C11, C12, C7, C8, C9: footprint component_tester:C0603 -> KiCad/Capacitors_SMD.pretty:C_0201
- C4, C5: footprint component_tester:C0805 -> KiCad/Capacitors_SMD.pretty:C_0805
- R1, R10, R11, R12, R13, R14, R16, R17, R18, R19, R2, R20, R3, R4, R5, R6, R7, R8, R9: footprint component_tester:R0805 -> KiCad/Resistors_SMD.pretty:R_0201
Changed lines of the file:
@@
 F 0 "C1" H 1900 3300 59  0000 L BNN
 F 1 "22p" H 2100 3100 59  0000 L BNN
-F 2 "component_tester:C0805" H 2000 3200 50  0001 C CNN
+F 2 "KiCad/Capacitors_SMD.pretty:C_0201" H 2000 3200 50  0001 C CNN
 F 3 "" H 2000 3200 50  0001 C CNN
 	1    2000 3200
@@
 F 0 "C2" H 1900 3900 59  0000 L BNN
 F 1 "22p" H 2100 3700 59  0000 L BNN
-F 2 "component_tester:C0805" H 2000 3800 50  0001 C CNN
+F 2 "KiCad/Capacitors_SMD.pretty:C_0201" H 2000 3800 50  0001 C CNN
 F 3 "" H 2000 3800 50  0001 C CNN
 	1    2000 3800
@@
 F 0 "R1" H 6750 3450 59  0001 L BNN
 F 1 "680" H 6750 3250 59  0001 L BNN
-F 2 "component_tester:R0805" H 6900 3400 50  0001 C CNN
+F 2 "KiCad/Resistors_SMD.pretty:R_0201" H 6900 3400 50  0001 C CNN
 F 3 "" H 6900 3400 50  0001 C CNN
 	1    6900 3400
@@
 F 0 "R2" H 6950 3450 59  0001 L BNN
 F 1 "470k" H 6950 3250 59  0001 L BNN
-F 2 "component_tester:R0805" H 7100 3400 50  0001 C CNN
+F 2 "KiCad/Resistors_SMD.pretty:R_0201" H 7100 3400 50  0001 C CNN
 F 3 "" H 7100 3400 50  0001 C CNN
 	1    7100 3400
@@
 F 0 "R3" H 7150 3450 59  0001 L BNN
 F 1 "680" H 7150 3250 59  0001 L BNN
-F 2 "component_tester:R0805" H 7300 3400 50  0001 C CNN
+F 2 "KiCad/Resistors_SMD.pretty:R_0201" H 7300 3400 50  0001 C CNN
 F 3 "" H 7300 3400 50  0001 C CNN
 	1    7300 3400
@@
 F 0 "R4" H 7350 3450 59  0001 L BNN
 F 1 "470k" H 7350 3250 59  0001 L BNN
-F 2 "component_tester:R0805" H 7500 3400 50  0001 C CNN
+F 2 "KiCad/Resistors_SMD.pretty:R_0201" H 7500 3400 50  0001 C CNN
 F 3 "" H 7500 3400 50  0001 C CNN
 	1    7500 3400
@@
 F 0 "R5" H 7550 3450 59  0001 L BNN
 F 1 "680" H 7550 3250 59  0001 L BNN
-F 2 "component_tester:R0805" H 7700 3400 50  0001 C CNN
+F 2 "KiCad/Resistors_SMD.pretty:R_0201" H 7700 3400 50  0001 C CNN
 F 3 "" H 7700 3400 50  0001 C CNN
 	1    7700 3400
@@
 F 0 "R6" H 7750 3450 59  0001 L BNN
 F 1 "470k" H 7750 3250 59  0001 L BNN
-F 2 "component_tester:R0805" H 7900 3400 50  0001 C CNN
+F 2 "KiCad/Resistors_SMD.pretty:R_0201" H 7900 3400 50  0001 C CNN
 F 3 "" H 7900 3400 50  0001 C CNN
 	1    7900 3400
@@
 F 0 "R7" H 2250 2850 59  0000 L BNN
 F 1 "10k" H 2250 2650 59  0000 L BNN
-F 2 "component_tester:R0805" H 2400 2800 50  0001 C CNN
+F 2 "KiCad/Resistors_SMD.pretty:R_0201" H 2400 2800 50  0001 C CNN
 F 3 "" H 2400 2800 50  0001 C CNN
 	1    2400 2800
@@
 F 0 "C3" H 2700 4600 59  0000 L BNN
 F 1 "1n" H 2900 4400 59  0000 L BNN
-F 2 "component_tester:C0805" H 2800 4500 50  0001 C CNN
+F 2 "KiCad/Capacitors_SMD.pretty:C_0201" H 2800 4500 50  0001 C CNN
 F 3 "" H 2800 4500 50  0001 C CNN
 	1    2800 4500
@@
 AR Path="/7513E83E99E27C05" Ref="C4"  Part="1"
 AR Path="/5B1C6B30/7513E83E99E27C05" Ref="C4"  Part="1"
-F 0 "C4" H 2800 7100 59  0001 L BNN
-F 1 "47u" H 3000 6900 59  0001 L BNN
-F 2 "component_tester:C0805" H 2900 7000 50  0001 C CNN
+F 0 "C4" V 2850 7150 59  0000 L BNN
+F 1 "47u" V 3075 7125 59  0000 L BNN
+F 2 "KiCad/Capacitors_SMD.pretty:C_0805" H 2900 7000 50  0001 C CNN
 F 3 "" H 2900 7000 50  0001 C CNN
 	1    2900 7000
@@
 F 0 "C5" H 5200 7300 59  0000 L BNN
 F 1 "47u" H 5400 7100 59  0000 L BNN
-F 2 "component_tester:C0805" H 5300 7200 50  0001 C CNN
+F 2 "KiCad/Capacitors_SMD.pretty:C_0805" H 5300 7200 50  0001 C CNN
 F 3 "" H 5300 7200 50  0001 C CNN
 	1    5300 7200
@@
 F 0 "R8" H 4850 6950 59  0000 L BNN
 F 1 "750k" H 4850 6750 59  0000 L BNN
-F 2 "component_tester:R0805" H 5000 6900 50  0001 C CNN
+F 2 "KiCad/Resistors_SMD.pretty:R_0201" H 5000 6900 50  0001 C CNN
 F 3 "" H 5000 6900 50  0001 C CNN
 	1    5000 6900
@@
 F 0 "R9" H 4850 7550 59  0000 L BNN
 F 1 "240k" H 4850 7350 59  0000 L BNN
-F 2 "component_tester:R0805" H 5000 7500 50  0001 C CNN
+F 2 "KiCad/Resistors_SMD.pretty:R_0201" H 5000 7500 50  0001 C CNN
 F 3 "" H 5000 7500 50  0001 C CNN
 	1    5000 7500
@@
 F 0 "R10" H 4050 5650 59  0000 L BNN
 F 1 "1M" H 4050 5450 59  0000 L BNN
-F 2 "component_tester:R0805" H 4200 5600 50  0001 C CNN
+F 2 "KiCad/Resistors_SMD.pretty:R_0201" H 4200 5600 50  0001 C CNN
 F 3 "" H 4200 5600 50  0001 C CNN
 	1    4200 5600
@@
 F 0 "R11" H 5650 2150 59  0001 L BNN
 F 1 "330k" H 5650 1950 59  0001 L BNN
-F 2 "component_tester:R0805" H 5800 2100 50  0001 C CNN
+F 2 "KiCad/Resistors_SMD.pretty:R_0201" H 5800 2100 50  0001 C CNN
 F 3 "" H 5800 2100 50  0001 C CNN
 	1    5800 2100
@@
 F 0 "C6" H 2400 4500 59  0000 L BNN
 F 1 "100n" H 2600 4300 59  0000 L BNN
-F 2 "component_tester:C0805" H 2500 4400 50  0001 C CNN
+F 2 "KiCad/Capacitors_SMD.pretty:C_0201" H 2500 4400 50  0001 C CNN
 F 3 "" H 2500 4400 50  0001 C CNN
 	1    2500 4400
@@
 F 0 "R12" H 4050 6250 59  0000 L BNN
 F 1 "10k" H 4050 6050 59  0000 L BNN
-F 2 "component_tester:R0805" H 4200 6200 50  0001 C CNN
+F 2 "KiCad/Resistors_SMD.pretty:R_0201" H 4200 6200 50  0001 C CNN
 F 3 "" H 4200 6200 50  0001 C CNN
 	1    4200 6200
@@
 F 0 "R13" H 6050 2150 59  0000 L BNN
 F 1 "10k" H 6050 1950 59  0000 L BNN
-F 2 "component_tester:R0805" H 6200 2100 50  0001 C CNN
+F 2 "KiCad/Resistors_SMD.pretty:R_0201" H 6200 2100 50  0001 C CNN
 F 3 "" H 6200 2100 50  0001 C CNN
 	1    6200 2100
@@
 F 0 "R14" H 5250 1550 59  0000 L BNN
 F 1 "47k" H 5250 1350 59  0000 L BNN
-F 2 "component_tester:R0805" H 5400 1500 50  0001 C CNN
+F 2 "KiCad/Resistors_SMD.pretty:R_0201" H 5400 1500 50  0001 C CNN
 F 3 "" H 5400 1500 50  0001 C CNN
 	1    5400 1500
@@
 F 0 "R16" H 6250 7150 59  0001 L BNN
 F 1 "10k" H 6250 6950 59  0001 L BNN
-F 2 "component_tester:R0805" H 6400 7100 50  0001 C CNN
+F 2 "KiCad/Resistors_SMD.pretty:R_0201" H 6400 7100 50  0001 C CNN
 F 3 "" H 6400 7100 50  0001 C CNN
 	1    6400 7100
@@
 F 0 "R17" H 1750 7250 59  0000 L BNN
 F 1 "10k" H 1750 7050 59  0000 L BNN
-F 2 "component_tester:R0805" H 1900 7200 50  0001 C CNN
+F 2 "KiCad/Resistors_SMD.pretty:R_0201" H 1900 7200 50  0001 C CNN
 F 3 "" H 1900 7200 50  0001 C CNN
 	1    1900 7200
@@
 F 0 "C7" H 7800 2300 59  0000 L BNN
 F 1 "V 3p" H 8000 2100 59  0000 L BNN
-F 2 "component_tester:C0603" H 7900 2200 50  0001 C CNN
+F 2 "KiCad/Capacitors_SMD.pretty:C_0201" H 7900 2200 50  0001 C CNN
 F 3 "" H 7900 2200 50  0001 C CNN
 	1    7900 2200
@@
 F 0 "C8" H 7800 2500 59  0000 L BNN
 F 1 "V 3p" H 8000 2300 59  0000 L BNN
-F 2 "component_tester:C0603" H 7900 2400 50  0001 C CNN
+F 2 "KiCad/Capacitors_SMD.pretty:C_0201" H 7900 2400 50  0001 C CNN
 F 3 "" H 7900 2400 50  0001 C CNN
 	1    7900 2400
@@
 F 0 "C9" H 7800 2700 59  0000 L BNN
 F 1 "V 3p" H 8000 2500 59  0000 L BNN
-F 2 "component_tester:C0603" H 7900 2600 50  0001 C CNN
+F 2 "KiCad/Capacitors_SMD.pretty:C_0201" H 7900 2600 50  0001 C CNN
 F 3 "" H 7900 2600 50  0001 C CNN
 	1    7900 2600
@@
 F 0 "C10" H 8000 3300 59  0000 L BNN
 F 1 "V 3p" H 8200 3100 59  0000 L BNN
-F 2 "component_tester:C0603" H 8100 3200 50  0001 C CNN
+F 2 "KiCad/Capacitors_SMD.pretty:C_0201" H 8100 3200 50  0001 C CNN
 F 3 "" H 8100 3200 50  0001 C CNN
 	1    8100 3200
@@
 F 0 "C11" H 8300 3300 59  0000 L BNN
 F 1 "V 3p" H 8500 3100 59  0000 L BNN
-F 2 "component_tester:C0603" H 8400 3200 50  0001 C CNN
+F 2 "KiCad/Capacitors_SMD.pretty:C_0201" H 8400 3200 50  0001 C CNN
 F 3 "" H 8400 3200 50  0001 C CNN
 	1    8400 3200
@@
 F 0 "C12" H 8600 3300 59  0000 L BNN
 F 1 "V 3p" H 8800 3100 59  0000 L BNN
-F 2 "component_tester:C0603" H 8700 3200 50  0001 C CNN
+F 2 "KiCad/Capacitors_SMD.pretty:C_0201" H 8700 3200 50  0001 C CNN
 F 3 "" H 8700 3200 50  0001 C CNN
 	1    8700 3200
@@
 F 0 "R18" H 3650 7550 59  0001 L BNN
 F 1 "10k" H 3650 7350 59  0001 L BNN
-F 2 "component_tester:R0805" H 3800 7500 50  0001 C CNN
+F 2 "KiCad/Resistors_SMD.pretty:R_0201" H 3800 7500 50  0001 C CNN
 F 3 "" H 3800 7500 50  0001 C CNN
 	1    3800 7500
@@
 F 0 "R19" H 6550 6650 59  0001 L BNN
 F 1 "10k" H 6550 6450 59  0001 L BNN
-F 2 "component_tester:R0805" H 6700 6600 50  0001 C CNN
+F 2 "KiCad/Resistors_SMD.pretty:R_0201" H 6700 6600 50  0001 C CNN
 F 3 "" H 6700 6600 50  0001 C CNN
 	1    6700 6600
@@
 F 0 "R20" H 5750 7150 59  0001 L BNN
 F 1 "10k" H 5750 6950 59  0001 L BNN
-F 2 "component_tester:R0805" H 5900 7100 50  0001 C CNN
+F 2 "KiCad/Resistors_SMD.pretty:R_0201" H 5900 7100 50  0001 C CNN
 F 3 "" H 5900 7100 50  0001 C CNN
 	1    5900 7100

Commit message: Switch atemega to smaller footprint
Parts:
- removed IC1: MEGA48/88/168-AU, component_tester:TQFP32-08, symbol component_tester-eagle-import:MEGA48_88_168-AU
- added IC1: ATmega328P-MMH, KiCad/Housings_DFN_QFN.pretty:QFN-28-1EP_4x4mm_Pitch0.4mm, symbol atmega48a-mmh:ATmega328P-MMH
Connections:
- wire segments 211 -> 209

Commit message: Add OLED footprint
Parts:
- added J?: Conn_01x30, symbol Connector_Generic:Conn_01x30
- BAT1: footprint component_tester:CR2032 -> StefanHamminga/SH_Batteries.pretty:Battery_Retainer_2032_BK-912
Changed lines of the file:
@@
 F 0 "BAT1" H 2700 7400 50  0001 C CNN
 F 1 "CR2032" H 2700 7400 50  0001 C CNN
-F 2 "component_tester:CR2032" H 2700 7400 50  0001 C CNN
+F 2 "StefanHamminga/SH_Batteries.pretty:Battery_Retainer_2032_BK-912" H 2700 7400 50  0001 C CNN
 F 3 "" H 2700 7400 50  0001 C CNN
 	1    2700 7400
@@
 Wire Wire Line
 	5900 5025 5900 5900
+$Comp
+L Connector_Generic:Conn_01x30 J?
+U 1 1 5B4AE6A8
+P 11025 3675
+F 0 "J?" H 11105 3667 50  0000 L CNN
+F 1 "Conn_01x30" H 11105 3576 50  0000 L CNN
+F 2 "" H 11025 3675 50  0001 C CNN
+F 3 "~" H 11025 3675 50  0001 C CNN
+	1    11025 3675
+	1    0    0    -1
+$EndComp
 $EndSCHEMATC

Commit message: Connect up test pads
Parts:
- removed TP1, TP2, TP3, TP4, TP5, TP6: SMD-PAD_0.2X0.2, component_tester:PAD_0.2X0.2, symbol component_tester-eagle-import:SMD-PAD_0.2X0.2
- removed X10, X3: P3, component_tester:STIFT_WINKL_SMD, symbol component_tester-eagle-import:STIFT_WINKL_SMD
- removed X11, X4: P1, component_tester:STIFT_WINKL_SMD, symbol component_tester-eagle-import:STIFT_WINKL_SMD
- removed X12, X5: P2, component_tester:STIFT_WINKL_SMD, symbol component_tester-eagle-import:STIFT_WINKL_SMD
- removed X2: P1, component_tester:STIFT, symbol component_tester-eagle-import:STIFT
- removed X7: P2, component_tester:STIFT, symbol component_tester-eagle-import:STIFT
- removed X8: P3, component_tester:STIFT, symbol component_tester-eagle-import:STIFT
- added DRAWING2: DRAWING, drawings:pads, symbol Connector_Generic:Conn_01x03
- added DRAWING3: DRAWING, drawings:pads_bottom, symbol Connector_Generic:Conn_01x03
- OLED1: renamed from J?; footprint (none) -> component_tester:SSD1306
Connections:
- net labels removed: SEG1, SEG2, SEG3
- wire segments 209 -> 210
Other:
- note removed: "Bedienteil"
- note removed: "Reserve"
