File: kicad/component_tester_1.sch (KiCad schematic (older format))
At the start: 51 parts, among them IC1 ATmega328P-MMH, IC2 MCP1640, Q1 8 MHz, SW1 TASTER-RACON8SMD, T1 BC847, T2 BSS123, T3 PMV65XP, T5 BSS84, X1 MICRO-USB, X6 ISP, X9 STIFTLEISTE_2,54MM_1X3_WI-SMD

Commit message: Sort out ground net
Connections:
- net labels removed: +
- wire segments 210 -> 215
Changed lines of the file:
@@
 Wire Wire Line
 	2900 7200 2900 7800
-Text GLabel 2900 7200 0    10   BiDi ~ 0
-GND
 Wire Wire Line
 	4300 7500 4300 7700
-Text GLabel 4300 7500 0    10   BiDi ~ 0
-GND
 Wire Wire Line
 	5900 7400 5900 7300
@@
 	2300 7100 2700 7100
 Connection ~ 2700 7100
-Text GLabel 2700 7200 0    10   BiDi ~ 0
-BAT+
 Wire Wire Line
 	1600 6400 2000 6400
@@
 	1    1400 6300
 	-1   0    0    1
-$EndComp
-$Comp
-L component_tester-eagle-import:CR2032 BAT1
-U 1 0 D31478EC87295480
-P 2700 7400
-AR Path="/D31478EC87295480" Ref="BAT1"  Part="1"
-AR Path="/5B1C6B30/D31478EC87295480" Ref="BAT1"  Part="1"
-F 0 "BAT1" H 2700 7400 50  0001 C CNN
-F 1 "CR2032" H 2700 7400 50  0001 C CNN
-F 2 "StefanHamminga/SH_Batteries.pretty:Battery_Retainer_2032_BK-912" H 2700 7400 50  0001 C CNN
-F 3 "" H 2700 7400 50  0001 C CNN
-	1    2700 7400
-	0    -1   -1   0
 $EndComp
 $Comp
@@
 Text Notes 725  725  0    127  ~ 0
 K.-H. Kübbeler, DF3DCB, DH8GHH
-Text GLabel 2600 7200 0    10   BiDi ~ 0
-+
 $Comp
 L atmega48a-mmh:ATmega328P-MMH IC1
@@
 $EndComp
 Wire Wire Line
-	4800 5075 4800 5250
-Wire Wire Line
 	3575 2625 3700 2625
 Wire Wire Line
@@
 Wire Wire Line
 	8500 950  8500 1375
+$Comp
+L component_tester-eagle-import:CR2032 BAT1
+U 1 0 D31478EC87295480
+P 2700 7400
+AR Path="/D31478EC87295480" Ref="BAT1"  Part="1"
+AR Path="/5B1C6B30/D31478EC87295480" Ref="BAT1"  Part="1"
+F 0 "BAT1" H 2700 7400 50  0001 C CNN
+F 1 "CR2032" H 2700 7400 50  0001 C CNN
+F 2 "StefanHamminga/SH_Batteries.pretty:Battery_Retainer_2032_BK-912" H 2700 7400 50  0001 C CNN
+F 3 "" H 2700 7400 50  0001 C CNN
+	1    2700 7400
+	0    -1   -1   0
+$EndComp
+Wire Wire Line
+	4800 5150 4650 5150
+Wire Wire Line
+	4650 5150 4650 5075
+Connection ~ 4800 5150
+Wire Wire Line
+	4800 5150 4800 5075
+Wire Wire Line
+	4500 5075 4500 5150
+Wire Wire Line
+	4500 5150 4650 5150
+Connection ~ 4650 5150
+Wire Wire Line
+	4800 5150 4800 5250
 $EndSCHEMATC

Commit message: Remove all the ground labels and zones
Changed lines of the file:
@@
 Wire Wire Line
 	2975 2925 3075 2925
-Text GLabel 2975 2925 0    10   BiDi ~ 0
-GND
 Wire Wire Line
 	2975 3525 3075 3525
-Text GLabel 2975 3525 0    10   BiDi ~ 0
-GND
 Wire Wire Line
 	875  1725 1275 1725
@@
 	1275 1525 1275 1725
 Connection ~ 1275 1725
-Text GLabel 875  1725 0    10   BiDi ~ 0
-GND
 Wire Wire Line
 	5400 7800 5300 7800
@@
 	5000 7800 5000 7700
 Connection ~ 5300 7800
-Text GLabel 5400 7800 0    10   BiDi ~ 0
-GND
 Wire Wire Line
 	7100 6800 7100 7200
-Text GLabel 7100 6800 0    10   BiDi ~ 0
-GND
 Wire Wire Line
 	5800 1425 5800 825
-Text GLabel 5800 1425 0    10   BiDi ~ 0
-GND
 Wire Wire Line
 	5400 1825 5400 1925
-Text GLabel 5400 1825 0    10   BiDi ~ 0
-GND
 Wire Wire Line
 	1700 6100 1700 6900
 Wire Wire Line
 	1600 6100 1700 6100
-Text GLabel 1700 6100 1    10   BiDi ~ 0
-GND
 Wire Wire Line
 	8600 4725 8900 4725
 Wire Wire Line
 	8900 4725 8900 5500
-Text GLabel 8600 4725 0    10   BiDi ~ 0
-GND
 Wire Wire Line
 	6400 7400 6400 7300
-Text GLabel 6400 7400 0    10   BiDi ~ 0
-GND
 Wire Wire Line
 	7700 1725 7600 1725
-Text GLabel 7700 1725 0    10   BiDi ~ 0
-GND
 Wire Wire Line
 	7700 1925 7600 1925
-Text GLabel 7700 1925 0    10   BiDi ~ 0
-GND
 Wire Wire Line
 	7700 2125 7600 2125
-Text GLabel 7700 2125 0    10   BiDi ~ 0
-GND
 Wire Wire Line
 	8100 2925 8100 3025
-Text GLabel 8100 2925 0    10   BiDi ~ 0
-GND
 Wire Wire Line
 	8400 2925 8400 3025
-Text GLabel 8400 2925 0    10   BiDi ~ 0
-GND
 Wire Wire Line
 	8700 2925 8700 3025
-Text GLabel 8700 2925 0    10   BiDi ~ 0
-GND
 Wire Wire Line
 	6200 5125 6200 5800
-Text GLabel 6200 5600 0    10   BiDi ~ 0
-GND
 Wire Wire Line
 	2700 7600 2700 7700
@@
 	1900 7700 2300 7700
 Connection ~ 2300 7700
-Text GLabel 2700 7600 0    10   BiDi ~ 0
-GND
 Wire Wire Line
 	2900 7200 2900 7800
@@
 Wire Wire Line
 	5900 7400 5900 7300
-Text GLabel 5900 7400 0    10   BiDi ~ 0
-GND
 Wire Wire Line
 	3375 2925 3575 2925
@@
 Connection ~ 1800 6500
 Connection ~ 1900 6500
-Text GLabel 1600 6500 1    10   BiDi ~ 0
-VCC
 Wire Wire Line
 	2700 7200 2700 7100
@@
 Wire Wire Line
 	8500 950  8500 1375
+Wire Wire Line
+	4800 5150 4650 5150
+Wire Wire Line
+	4650 5150 4650 5075
+Connection ~ 4800 5150
+Wire Wire Line
+	4800 5150 4800 5075
+Wire Wire Line
+	4500 5075 4500 5150
+Wire Wire Line
+	4500 5150 4650 5150
+Connection ~ 4650 5150
+Wire Wire Line
+	4800 5150 4800 5250
 $Comp
 L component_tester-eagle-import:CR2032 BAT1
 U 1 0 D31478EC87295480
-P 2700 7400
+P 2650 8075
 AR Path="/D31478EC87295480" Ref="BAT1"  Part="1"
 AR Path="/5B1C6B30/D31478EC87295480" Ref="BAT1"  Part="1"
-F 0 "BAT1" H 2700 7400 50  0001 C CNN
-F 1 "CR2032" H 2700 7400 50  0001 C CNN
-F 2 "StefanHamminga/SH_Batteries.pretty:Battery_Retainer_2032_BK-912" H 2700 7400 50  0001 C CNN
-F 3 "" H 2700 7400 50  0001 C CNN
-	1    2700 7400
-	0    -1   -1   0
-$EndComp
-Wire Wire Line
-	4800 5150 4650 5150
-Wire Wire Line
-	4650 5150 4650 5075
-Connection ~ 4800 5150
-Wire Wire Line
-	4800 5150 4800 5075
-Wire Wire Line
-	4500 5075 4500 5150
-Wire Wire Line
-	4500 5150 4650 5150
-Connection ~ 4650 5150
-Wire Wire Line
-	4800 5150 4800 5250
+F 0 "BAT1" H 2650 8075 50  0001 C CNN
+F 1 "CR2032" H 2650 8075 50  0001 C CNN
+F 2 "StefanHamminga/SH_Batteries.pretty:Battery_Retainer_2032_BK-912" H 2650 8075 50  0001 C CNN
+F 3 "" H 2650 8075 50  0001 C CNN
+	1    2650 8075
+	0    -1   -1   0
+$EndComp
 $EndSCHEMATC

Commit message: Sort out power nets/labels
Connections:
- net labels added: +BATT
- net labels removed: BAT+
- wire segments 215 -> 216
Changed lines of the file:
@@
 	1275 1225 1275 1025
 Connection ~ 1275 1025
-Text Label 3000 3525 0    10   ~ 0
-+5V
 Wire Wire Line
 	2250 2375 2750 2375
-Text Label 2250 2375 0    10   ~ 0
-+5V
 Wire Wire Line
 	5400 725  5400 825
-Text Label 5400 725  0    10   ~ 0
-+5V
 Wire Wire Line
 	6200 725  6200 1425
-Text Label 6200 725  0    10   ~ 0
-+5V
 Wire Wire Line
 	5300 6500 5500 6500
@@
 Connection ~ 5300 6500
 Connection ~ 5000 6500
-Text Label 5300 6500 0    10   ~ 0
-+5V
 Wire Wire Line
 	8600 4525 8900 4525
 Wire Wire Line
 	8900 4525 8900 4225
-Text Label 8600 4525 0    10   ~ 0
-+5V
 Wire Wire Line
 	3150 2375 3350 2375
@@
 	1    1275 1325
 	1    0    0    -1
-$EndComp
-$Comp
-L component_tester-eagle-import:+5V #+5V7
-U 1 0 BC662C5A60B97BFF
-P 2200 7100
-AR Path="/BC662C5A60B97BFF" Ref="#+5V7"  Part="1"
-AR Path="/5B1C6B30/BC662C5A60B97BFF" Ref="#+5V07"  Part="1"
-F 0 "#+5V07" H 2200 7100 50  0001 C CNN
-F 1 "BAT+" V 2100 6900 59  0000 L BNN
-F 2 "" H 2200 7100 50  0001 C CNN
-F 3 "" H 2200 7100 50  0001 C CNN
-	1    2200 7100
-	0    -1   -1   0
 $EndComp
 $Comp
@@
 L component_tester-eagle-import:CR2032 BAT1
 U 1 0 D31478EC87295480
-P 2650 8075
+P 2700 7400
 AR Path="/D31478EC87295480" Ref="BAT1"  Part="1"
 AR Path="/5B1C6B30/D31478EC87295480" Ref="BAT1"  Part="1"
-F 0 "BAT1" H 2650 8075 50  0001 C CNN
-F 1 "CR2032" H 2650 8075 50  0001 C CNN
-F 2 "StefanHamminga/SH_Batteries.pretty:Battery_Retainer_2032_BK-912" H 2650 8075 50  0001 C CNN
-F 3 "" H 2650 8075 50  0001 C CNN
-	1    2650 8075
+F 0 "BAT1" H 2700 7400 50  0001 C CNN
+F 1 "CR2032" H 2700 7400 50  0001 C CNN
+F 2 "StefanHamminga/SH_Batteries.pretty:Battery_Retainer_2032_BK-912" H 2700 7400 50  0001 C CNN
+F 3 "" H 2700 7400 50  0001 C CNN
+	1    2700 7400
 	0    -1   -1   0
 $EndComp
@@
 	1    0    0    -1
 $EndComp
+$Comp
+L power:+BATT #PWR0101
+U 1 1 5B66E8BE
+P 2300 7000
+F 0 "#PWR0101" H 2300 6850 50  0001 C CNN
+F 1 "+BATT" H 2315 7173 50  0000 C CNN
+F 2 "" H 2300 7000 50  0001 C CNN
+F 3 "" H 2300 7000 50  0001 C CNN
+	1    2300 7000
+	1    0    0    -1
+$EndComp
+Wire Wire Line
+	2300 7100 2300 7000
 $EndSCHEMATC

Commit message: Delete some connectors
Parts:
- removed X9: STIFTLEISTE_2,54MM_1X3_WI-SMD, component_tester:STIFTLEISTE_2,54MM_1X3_WI-SMD, symbol component_tester-eagle-import:STIFTLEISTE_2,54MM_1X3_WI-SMD
Connections:
- wire segments 216 -> 213
Changed lines of the file:
@@
 	8100 1725 8100 1525
-Wire Wire Line
-	8100 2325 9000 2325
 Wire Wire Line
 	8000 1725 8100 1725
@@
 	8400 2425 8400 1925
 Wire Wire Line
-	8400 2425 9000 2425
-Wire Wire Line
 	8000 1925 8400 1925
 Wire Wire Line
@@
 Wire Wire Line
 	8700 2125 8700 2525
-Wire Wire Line
-	8700 2525 9000 2525
 Wire Wire Line
 	8000 2125 8700 2125
@@
 AR Path="/CB1356D799561180" Ref="R11"  Part="1"
 AR Path="/5B1C6B30/CB1356D799561180" Ref="R11"  Part="1"
-F 0 "R11" H 5650 1675 59  0001 L BNN
-F 1 "330k" H 5650 1475 59  0001 L BNN
+F 0 "R11" H 5650 1675 59  0000 L BNN
+F 1 "330k" H 5650 1475 59  0000 L BNN
 F 2 "KiCad/Resistors_SMD.pretty:R_0201" H 5800 1625 50  0001 C CNN
 F 3 "" H 5800 1625 50  0001 C CNN
@@
 	1    7500 1725
 	0    1    1    0
-$EndComp
-$Comp
-L component_tester-eagle-import:STIFTLEISTE_2,54MM_1X3_WI-SMD X9
-U 1 0 E2DA910908FA697E
-P 9000 2425
-AR Path="/E2DA910908FA697E" Ref="X9"  Part="1"
-AR Path="/5B1C6B30/E2DA910908FA697E" Ref="X9"  Part="1"
-F 0 "X9" H 8950 2575 42  0001 L BNN
-F 1 "STIFTLEISTE_2,54MM_1X3_WI-SMD" H 8950 2225 42  0001 L BNN
-F 2 "component_tester:STIFTLEISTE_2,54MM_1X3_WI-SMD" H 9000 2425 50  0001 C CNN
-F 3 "" H 9000 2425 50  0001 C CNN
-	1    9000 2425
-	1    0    0    -1
 $EndComp
 $Comp
@@
 U 1 1 5B4B01B0
 P 8400 750
-F 0 "DRAWING2" H 8480 792 50  0000 L CNN
-F 1 "DRAWING" H 8480 701 50  0000 L CNN
+F 0 "DRAWING2" V 8350 950 50  0000 L CNN
+F 1 "DRAWING" V 8425 1000 50  0000 L CNN
 F 2 "drawings:pads" H 8400 750 50  0001 C CNN
 F 3 "~" H 8400 750 50  0001 C CNN
@@
 U 1 1 5B4B01B7
 P 8400 1175
-F 0 "DRAWING3" H 8480 1217 50  0000 L CNN
-F 1 "DRAWING" H 8480 1126 50  0000 L CNN
+F 0 "DRAWING3" V 8375 1450 50  0000 L CNN
+F 1 "DRAWING" V 8450 1500 50  0000 L CNN
 F 2 "drawings:pads_bottom" H 8400 1175 50  0001 C CNN
 F 3 "~" H 8400 1175 50  0001 C CNN

Commit message: Import Adafruit OLED breakout
Parts:
- removed OLED1: Conn_01x30, component_tester:SSD1306, symbol Connector_Generic:Conn_01x30
- renumbered BAT1 to BAT201, C15 to C201, C6 to C202, C4 to C203, C1 to C204, C2 to C205, C3 to C206, C5 to C207, C7 to C208, C8 to C209, C9 to C210, C10 to C211, C11 to C212, C12 to C213, D2 to D201, D1 to D202, D5 to D203, DRAWING2 to DRAWING201, DRAWING3 to DRAWING202, IC2 to IC201, IC1 to IC202, L1 to L201, Q1 to Q201, R17 to R201, R7 to R202, R18 to R203, R10 to R204, R12 to R205, R8 to R206, R9 to R207, R14 to R208, R11 to R209, R20 to R210, R13 to R211, R16 to R212, R19 to R213, R1 to R214, R2 to R215, R3 to R216, R4 to R217, R5 to R218, R6 to R219, SW1 to SW201, T3 to T201, T5 to T202, T2 to T203, T1 to T204, X1 to X201, X6 to X202

Commit message: Switch 0201 footprints for 0402
Parts:
- C202, C204, C205, C206, C208, C209, C210, C211, C212, C213: footprint KiCad/Capacitors_SMD.pretty:C_0201 -> KiCad/Capacitors_SMD.pretty:C_0402
- R201, R202, R203, R204, R205, R206, R207, R208, R209, R210, R211, R212, R213, R214, R215, R216, R217, R218, R219: footprint KiCad/Resistors_SMD.pretty:R_0201 -> KiCad/Resistors_SMD.pretty:R_0402
Changed lines of the file:
@@
 F 0 "C204" H 3075 3025 59  0000 L BNN
 F 1 "22p" H 3275 2825 59  0000 L BNN
-F 2 "KiCad/Capacitors_SMD.pretty:C_0201" H 3175 2925 50  0001 C CNN
+F 2 "KiCad/Capacitors_SMD.pretty:C_0402" H 3175 2925 50  0001 C CNN
 F 3 "" H 3175 2925 50  0001 C CNN
 	1    3175 2925
@@
 F 0 "C205" H 3075 3625 59  0000 L BNN
 F 1 "22p" H 3275 3425 59  0000 L BNN
-F 2 "KiCad/Capacitors_SMD.pretty:C_0201" H 3175 3525 50  0001 C CNN
+F 2 "KiCad/Capacitors_SMD.pretty:C_0402" H 3175 3525 50  0001 C CNN
 F 3 "" H 3175 3525 50  0001 C CNN
 	1    3175 3525
@@
 F 0 "R214" H 6750 2975 59  0001 L BNN
 F 1 "680" H 6750 2775 59  0001 L BNN
-F 2 "KiCad/Resistors_SMD.pretty:R_0201" H 6900 2925 50  0001 C CNN
+F 2 "KiCad/Resistors_SMD.pretty:R_0402" H 6900 2925 50  0001 C CNN
 F 3 "" H 6900 2925 50  0001 C CNN
 	1    6900 2925
@@
 F 0 "R215" H 6950 2975 59  0001 L BNN
 F 1 "470k" H 6950 2775 59  0001 L BNN
-F 2 "KiCad/Resistors_SMD.pretty:R_0201" H 7100 2925 50  0001 C CNN
+F 2 "KiCad/Resistors_SMD.pretty:R_0402" H 7100 2925 50  0001 C CNN
 F 3 "" H 7100 2925 50  0001 C CNN
 	1    7100 2925
@@
 F 0 "R216" H 7150 2975 59  0001 L BNN
 F 1 "680" H 7150 2775 59  0001 L BNN
-F 2 "KiCad/Resistors_SMD.pretty:R_0201" H 7300 2925 50  0001 C CNN
+F 2 "KiCad/Resistors_SMD.pretty:R_0402" H 7300 2925 50  0001 C CNN
 F 3 "" H 7300 2925 50  0001 C CNN
 	1    7300 2925
@@
 F 0 "R217" H 7350 2975 59  0001 L BNN
 F 1 "470k" H 7350 2775 59  0001 L BNN
-F 2 "KiCad/Resistors_SMD.pretty:R_0201" H 7500 2925 50  0001 C CNN
+F 2 "KiCad/Resistors_SMD.pretty:R_0402" H 7500 2925 50  0001 C CNN
 F 3 "" H 7500 2925 50  0001 C CNN
 	1    7500 2925
@@
 F 0 "R218" H 7550 2975 59  0001 L BNN
 F 1 "680" H 7550 2775 59  0001 L BNN
-F 2 "KiCad/Resistors_SMD.pretty:R_0201" H 7700 2925 50  0001 C CNN
+F 2 "KiCad/Resistors_SMD.pretty:R_0402" H 7700 2925 50  0001 C CNN
 F 3 "" H 7700 2925 50  0001 C CNN
 	1    7700 2925
@@
 F 0 "R219" H 7750 2975 59  0001 L BNN
 F 1 "470k" H 7750 2775 59  0001 L BNN
-F 2 "KiCad/Resistors_SMD.pretty:R_0201" H 7900 2925 50  0001 C CNN
+F 2 "KiCad/Resistors_SMD.pretty:R_0402" H 7900 2925 50  0001 C CNN
 F 3 "" H 7900 2925 50  0001 C CNN
 	1    7900 2925
@@
 $EndComp
 $Comp
-L component_tester-eagle-import:GND #GND0201
+L component_tester-eagle-import:GND #GND0402
 U 1 0 714A278CA07C0193
 P 775 1725
-F 0 "#GND0201" H 775 1725 50  0001 C CNN
+F 0 "#GND0402" H 775 1725 50  0001 C CNN
 F 1 "GND" H 675 1625 59  0000 L BNN
 F 2 "" H 775 1725 50  0001 C CNN
@@
 F 0 "R202" H 2800 2425 59  0000 L BNN
 F 1 "10k" H 2800 2225 59  0000 L BNN
-F 2 "KiCad/Resistors_SMD.pretty:R_0201" H 2950 2375 50  0001 C CNN
+F 2 "KiCad/Resistors_SMD.pretty:R_0402" H 2950 2375 50  0001 C CNN
 F 3 "" H 2950 2375 50  0001 C CNN
 	1    2950 2375
@@
 $EndComp
 $Comp
-L component_tester-eagle-import:+5V #+5V0201
+L component_tester-eagle-import:+5V #+5V0402
 U 1 0 AFC6B6985F6C2C2A
 P 675 1025
-F 0 "#+5V0201" H 675 1025 50  0001 C CNN
+F 0 "#+5V0402" H 675 1025 50  0001 C CNN
 F 1 "+5V" V 575 825 59  0000 L BNN
 F 2 "" H 675 1025 50  0001 C CNN
@@
 F 0 "C206" H 3700 2725 59  0000 L BNN
 F 1 "1n" H 3900 2525 59  0000 L BNN
-F 2 "KiCad/Capacitors_SMD.pretty:C_0201" H 3800 2625 50  0001 C CNN
+F 2 "KiCad/Capacitors_SMD.pretty:C_0402" H 3800 2625 50  0001 C CNN
 F 3 "" H 3800 2625 50  0001 C CNN
 	1    3800 2625
@@
 F 0 "R206" H 4850 6950 59  0000 L BNN
 F 1 "750k" H 4850 6750 59  0000 L BNN
-F 2 "KiCad/Resistors_SMD.pretty:R_0201" H 5000 6900 50  0001 C CNN
+F 2 "KiCad/Resistors_SMD.pretty:R_0402" H 5000 6900 50  0001 C CNN
 F 3 "" H 5000 6900 50  0001 C CNN
 	1    5000 6900
@@
 F 0 "R207" H 4850 7550 59  0000 L BNN
 F 1 "240k" H 4850 7350 59  0000 L BNN
-F 2 "KiCad/Resistors_SMD.pretty:R_0201" H 5000 7500 50  0001 C CNN
+F 2 "KiCad/Resistors_SMD.pretty:R_0402" H 5000 7500 50  0001 C CNN
 F 3 "" H 5000 7500 50  0001 C CNN
 	1    5000 7500
@@
 F 0 "R204" H 4050 5650 59  0000 L BNN
 F 1 "1M" H 4050 5450 59  0000 L BNN
-F 2 "KiCad/Resistors_SMD.pretty:R_0201" H 4200 5600 50  0001 C CNN
+F 2 "KiCad/Resistors_SMD.pretty:R_0402" H 4200 5600 50  0001 C CNN
 F 3 "" H 4200 5600 50  0001 C CNN
 	1    4200 5600
@@
 F 0 "R209" H 5650 1675 59  0000 L BNN
 F 1 "330k" H 5650 1475 59  0000 L BNN
-F 2 "KiCad/Resistors_SMD.pretty:R_0201" H 5800 1625 50  0001 C CNN
+F 2 "KiCad/Resistors_SMD.pretty:R_0402" H 5800 1625 50  0001 C CNN
 F 3 "" H 5800 1625 50  0001 C CNN
 	1    5800 1625
@@
 F 0 "C202" H 1475 1525 59  0000 L BNN
 F 1 "100n" H 1675 1325 59  0000 L BNN
-F 2 "KiCad/Capacitors_SMD.pretty:C_0201" H 1575 1425 50  0001 C CNN
+F 2 "KiCad/Capacitors_SMD.pretty:C_0402" H 1575 1425 50  0001 C CNN
 F 3 "" H 1575 1425 50  0001 C CNN
 	1    1575 1425
@@
 F 0 "R205" H 4050 6250 59  0000 L BNN
 F 1 "10k" H 4050 6050 59  0000 L BNN
-F 2 "KiCad/Resistors_SMD.pretty:R_0201" H 4200 6200 50  0001 C CNN
+F 2 "KiCad/Resistors_SMD.pretty:R_0402" H 4200 6200 50  0001 C CNN
 F 3 "" H 4200 6200 50  0001 C CNN
 	1    4200 6200
@@
 F 0 "R211" H 6050 1675 59  0000 L BNN
 F 1 "10k" H 6050 1475 59  0000 L BNN
-F 2 "KiCad/Resistors_SMD.pretty:R_0201" H 6200 1625 50  0001 C CNN
+F 2 "KiCad/Resistors_SMD.pretty:R_0402" H 6200 1625 50  0001 C CNN
 F 3 "" H 6200 1625 50  0001 C CNN
 	1    6200 1625
@@
 F 0 "R208" H 5250 1075 59  0000 L BNN
 F 1 "47k" H 5250 875 59  0000 L BNN
-F 2 "KiCad/Resistors_SMD.pretty:R_0201" H 5400 1025 50  0001 C CNN
+F 2 "KiCad/Resistors_SMD.pretty:R_0402" H 5400 1025 50  0001 C CNN
 F 3 "" H 5400 1025 50  0001 C CNN
 	1    5400 1025
@@
 F 0 "R212" H 6250 7150 59  0001 L BNN
 F 1 "10k" H 6250 6950 59  0001 L BNN
-F 2 "KiCad/Resistors_SMD.pretty:R_0201" H 6400 7100 50  0001 C CNN
+F 2 "KiCad/Resistors_SMD.pretty:R_0402" H 6400 7100 50  0001 C CNN
 F 3 "" H 6400 7100 50  0001 C CNN
 	1    6400 7100
@@
 F 0 "R201" H 1750 7250 59  0000 L BNN
 F 1 "10k" H 1750 7050 59  0000 L BNN
-F 2 "KiCad/Resistors_SMD.pretty:R_0201" H 1900 7200 50  0001 C CNN
+F 2 "KiCad/Resistors_SMD.pretty:R_0402" H 1900 7200 50  0001 C CNN
 F 3 "" H 1900 7200 50  0001 C CNN
 	1    1900 7200
@@
 F 0 "C208" H 7800 1825 59  0000 L BNN
 F 1 "V 3p" H 8000 1625 59  0000 L BNN
-F 2 "KiCad/Capacitors_SMD.pretty:C_0201" H 7900 1725 50  0001 C CNN
+F 2 "KiCad/Capacitors_SMD.pretty:C_0402" H 7900 1725 50  0001 C CNN
 F 3 "" H 7900 1725 50  0001 C CNN
 	1    7900 1725
@@
 F 0 "C209" H 7800 2025 59  0000 L BNN
 F 1 "V 3p" H 8000 1825 59  0000 L BNN
-F 2 "KiCad/Capacitors_SMD.pretty:C_0201" H 7900 1925 50  0001 C CNN
+F 2 "KiCad/Capacitors_SMD.pretty:C_0402" H 7900 1925 50  0001 C CNN
 F 3 "" H 7900 1925 50  0001 C CNN
 	1    7900 1925
@@
 F 0 "C210" H 7800 2225 59  0000 L BNN
 F 1 "V 3p" H 8000 2025 59  0000 L BNN
-F 2 "KiCad/Capacitors_SMD.pretty:C_0201" H 7900 2125 50  0001 C CNN
+F 2 "KiCad/Capacitors_SMD.pretty:C_0402" H 7900 2125 50  0001 C CNN
 F 3 "" H 7900 2125 50  0001 C CNN
 	1    7900 2125
@@
 F 0 "C211" H 8000 2825 59  0000 L BNN
 F 1 "V 3p" H 8200 2625 59  0000 L BNN
-F 2 "KiCad/Capacitors_SMD.pretty:C_0201" H 8100 2725 50  0001 C CNN
+F 2 "KiCad/Capacitors_SMD.pretty:C_0402" H 8100 2725 50  0001 C CNN
 F 3 "" H 8100 2725 50  0001 C CNN
 	1    8100 2725
@@
 F 0 "C212" H 8300 2825 59  0000 L BNN
 F 1 "V 3p" H 8500 2625 59  0000 L BNN
-F 2 "KiCad/Capacitors_SMD.pretty:C_0201" H 8400 2725 50  0001 C CNN
+F 2 "KiCad/Capacitors_SMD.pretty:C_0402" H 8400 2725 50  0001 C CNN
 F 3 "" H 8400 2725 50  0001 C CNN
 	1    8400 2725
@@
 F 0 "C213" H 8600 2825 59  0000 L BNN
 F 1 "V 3p" H 8800 2625 59  0000 L BNN
-F 2 "KiCad/Capacitors_SMD.pretty:C_0201" H 8700 2725 50  0001 C CNN
+F 2 "KiCad/Capacitors_SMD.pretty:C_0402" H 8700 2725 50  0001 C CNN
 F 3 "" H 8700 2725 50  0001 C CNN
 	1    8700 2725
@@
 F 0 "R203" H 3650 7550 59  0001 L BNN
 F 1 "10k" H 3650 7350 59  0001 L BNN
-F 2 "KiCad/Resistors_SMD.pretty:R_0201" H 3800 7500 50  0001 C CNN
+F 2 "KiCad/Resistors_SMD.pretty:R_0402" H 3800 7500 50  0001 C CNN
 F 3 "" H 3800 7500 50  0001 C CNN
 	1    3800 7500
@@
 $EndComp
 $Comp
-L component_tester-eagle-import:VCC #P+0201
+L component_tester-eagle-import:VCC #P+0402
 U 1 0 93600057BCDF72C5
 P 1800 5300
-F 0 "#P+0201" H 1800 5300 50  0001 C CNN
+F 0 "#P+0402" H 1800 5300 50  0001 C CNN
 F 1 "VCC" V 1700 5200 59  0000 L BNN
 F 2 "" H 1800 5300 50  0001 C CNN
@@
 F 0 "R213" H 6550 6650 59  0001 L BNN
 F 1 "10k" H 6550 6450 59  0001 L BNN
-F 2 "KiCad/Resistors_SMD.pretty:R_0201" H 6700 6600 50  0001 C CNN
+F 2 "KiCad/Resistors_SMD.pretty:R_0402" H 6700 6600 50  0001 C CNN
 F 3 "" H 6700 6600 50  0001 C CNN
 	1    6700 6600
@@
 F 0 "R210" H 5750 7150 59  0001 L BNN
 F 1 "10k" H 5750 6950 59  0001 L BNN
-F 2 "KiCad/Resistors_SMD.pretty:R_0201" H 5900 7100 50  0001 C CNN
+F 2 "KiCad/Resistors_SMD.pretty:R_0402" H 5900 7100 50  0001 C CNN
 F 3 "" H 5900 7100 50  0001 C CNN
 	1    5900 7100

Commit message: Switch button footprint
Parts:
- Q201: footprint component_tester:HC49UP -> KiCad/Crystals.pretty:Crystal_SMD_Abracon_ABM3-2pin_5.0x3.2mm
- SW201: value TASTER-RACON8SMD -> Tactile Switch; footprint component_tester:TASTER-RACON8SMD -> smisioto.eu/kicad_libs/modules/w_switch.pretty:smd_push2
Changed lines of the file:
@@
 F 0 "Q201" H 3625 3225 42  0000 L BNN
 F 1 "8 MHz" H 3625 2975 42  0000 L BNN
-F 2 "component_tester:HC49UP" H 3475 3225 50  0001 C CNN
+F 2 "KiCad/Crystals.pretty:Crystal_SMD_Abracon_ABM3-2pin_5.0x3.2mm" H 3475 3225 50  0001 C CNN
 F 3 "" H 3475 3225 50  0001 C CNN
 	1    3475 3225
@@
 U 1 0 9A392703E9E31E47
 P 5200 5900
-F 0 "SW201" H 4980 6090 59  0001 L BNN
-F 1 "TASTER-RACON8SMD" H 4950 5680 59  0001 L BNN
-F 2 "component_tester:TASTER-RACON8SMD" H 5200 5900 50  0001 C CNN
+F 0 "SW201" H 4980 6090 59  0000 L BNN
+F 1 "Tactile Switch" H 4950 5680 59  0001 L BNN
+F 2 "smisioto.eu/kicad_libs/modules/w_switch.pretty:smd_push2" H 5200 5900 50  0001 C CNN
 F 3 "" H 5200 5900 50  0001 C CNN
 	1    5200 5900
