File: kicad/component_tester_1.sch (KiCad schematic (older format))
At the start: 49 parts, among them IC201 MCP1640, IC202 ATmega328P-MMH, Q201 8 MHz, SW201 EVQ, T201 PMV65XP, T202 BSS84, T203 BSS123, T204 BC847, X201 MICRO-USB, X202 ISP

Commit message: Work on placing components
Parts:
- removed L201: 4,7 uH, component_tester:L1210, symbol component_tester-eagle-import:L1210
- added L201: 4.7uH, KiCad/Resistors_SMD.pretty:R_0603, symbol pspice:INDUCTOR
- Q201: footprint KiCad/Crystals.pretty:Crystal_SMD_Abracon_ABM3-2pin_5.0x3.2mm -> mcous/kicad-lib/footprints/crystal.pretty:NDK-NX3225GA_xtal
Changed lines of the file:
@@
 	4300 6975 4300 6875
-Wire Wire Line
-	4300 6875 4100 6875
 Wire Wire Line
 	5000 7675 5000 7575
@@
 Wire Wire Line
 	3300 5925 3300 5675
-Wire Wire Line
-	3700 6875 3300 6875
 Wire Wire Line
 	3300 6875 3300 6575
@@
 F 0 "Q201" V 3500 3325 42  0000 L BNN
 F 1 "8 MHz" H 3625 2975 42  0000 L BNN
-F 2 "KiCad/Crystals.pretty:Crystal_SMD_Abracon_ABM3-2pin_5.0x3.2mm" H 3475 3225 50  0001 C CNN
+F 2 "mcous/kicad-lib/footprints/crystal.pretty:NDK-NX3225GA_xtal" H 3475 3225 50  0001 C CNN
 F 3 "" H 3475 3225 50  0001 C CNN
 	1    3475 3225
@@
 F 3 "" H 4300 7375 50  0001 C CNN
 	1    4300 7375
-	1    0    0    -1
-$EndComp
-$Comp
-L component_tester-eagle-import:L1210 L201
-U 1 0 F60B72F86BE0507A
-P 3900 6875
-F 0 "L201" H 3875 6975 42  0000 L BNN
-F 1 "4,7 uH" H 3800 6725 42  0000 L BNN
-F 2 "component_tester:L1210" H 3900 6875 50  0001 C CNN
-F 3 "" H 3900 6875 50  0001 C CNN
-	1    3900 6875
 	1    0    0    -1
 $EndComp
@@
 Wire Wire Line
 	5900 5650 5900 5925
+$Comp
+L pspice:INDUCTOR L201
+U 1 1 5B2621E0
+P 3875 6875
+F 0 "L201" H 3875 7090 50  0000 C CNN
+F 1 "4.7uH" H 3875 6999 50  0000 C CNN
+F 2 "KiCad/Resistors_SMD.pretty:R_0603" H 3875 6875 50  0001 C CNN
+F 3 "" H 3875 6875 50  0001 C CNN
+	1    3875 6875
+	1    0    0    -1
+$EndComp
+Wire Wire Line
+	3300 6875 3625 6875
+Wire Wire Line
+	4300 6875 4125 6875
 $EndSCHEMATC

Commit message: Switch back to 0201s and continue placing
Parts:
- C202, C204, C205, C206, C208, C209, C210, C211, C212, C213: footprint KiCad/Capacitors_SMD.pretty:C_0402 -> KiCad/Capacitors_SMD.pretty:C_0201
- R201, R202, R203, R204, R205, R206, R207, R208, R209, R210, R211, R212, R213, R214, R215, R216, R217, R218, R219: footprint KiCad/Resistors_SMD.pretty:R_0402 -> KiCad/Resistors_SMD.pretty:R_0201
Changed lines of the file:
@@
 F 0 "C204" H 3075 3025 59  0000 L BNN
 F 1 "22p" H 3275 2825 59  0000 L BNN
-F 2 "KiCad/Capacitors_SMD.pretty:C_0402" H 3175 2925 50  0001 C CNN
+F 2 "KiCad/Capacitors_SMD.pretty:C_0201" H 3175 2925 50  0001 C CNN
 F 3 "" H 3175 2925 50  0001 C CNN
 	1    3175 2925
@@
 F 0 "C205" H 3075 3625 59  0000 L BNN
 F 1 "22p" H 3275 3425 59  0000 L BNN
-F 2 "KiCad/Capacitors_SMD.pretty:C_0402" H 3175 3525 50  0001 C CNN
+F 2 "KiCad/Capacitors_SMD.pretty:C_0201" H 3175 3525 50  0001 C CNN
 F 3 "" H 3175 3525 50  0001 C CNN
 	1    3175 3525
@@
 F 0 "R214" H 6750 2975 59  0000 L BNN
 F 1 "680" H 6550 2975 59  0000 L BNN
-F 2 "KiCad/Resistors_SMD.pretty:R_0402" H 6900 2925 50  0001 C CNN
+F 2 "KiCad/Resistors_SMD.pretty:R_0201" H 6900 2925 50  0001 C CNN
 F 3 "" H 6900 2925 50  0001 C CNN
 	1    6900 2925
@@
 F 0 "R215" H 7000 2975 59  0000 L BNN
 F 1 "470k" H 6725 2950 59  0000 L BNN
-F 2 "KiCad/Resistors_SMD.pretty:R_0402" H 7100 2925 50  0001 C CNN
+F 2 "KiCad/Resistors_SMD.pretty:R_0201" H 7100 2925 50  0001 C CNN
 F 3 "" H 7100 2925 50  0001 C CNN
 	1    7100 2925
@@
 F 0 "R216" H 7150 2975 59  0000 L BNN
 F 1 "680" H 6950 2975 59  0000 L BNN
-F 2 "KiCad/Resistors_SMD.pretty:R_0402" H 7300 2925 50  0001 C CNN
+F 2 "KiCad/Resistors_SMD.pretty:R_0201" H 7300 2925 50  0001 C CNN
 F 3 "" H 7300 2925 50  0001 C CNN
 	1    7300 2925
@@
 F 0 "R217" H 7350 2975 59  0000 L BNN
 F 1 "470k" H 7125 2950 59  0000 L BNN
-F 2 "KiCad/Resistors_SMD.pretty:R_0402" H 7500 2925 50  0001 C CNN
+F 2 "KiCad/Resistors_SMD.pretty:R_0201" H 7500 2925 50  0001 C CNN
 F 3 "" H 7500 2925 50  0001 C CNN
 	1    7500 2925
@@
 F 0 "R218" H 7550 2975 59  0000 L BNN
 F 1 "680" H 7350 2975 59  0000 L BNN
-F 2 "KiCad/Resistors_SMD.pretty:R_0402" H 7700 2925 50  0001 C CNN
+F 2 "KiCad/Resistors_SMD.pretty:R_0201" H 7700 2925 50  0001 C CNN
 F 3 "" H 7700 2925 50  0001 C CNN
 	1    7700 2925
@@
 F 0 "R219" H 7750 2975 59  0000 L BNN
 F 1 "470k" H 7525 2950 59  0000 L BNN
-F 2 "KiCad/Resistors_SMD.pretty:R_0402" H 7900 2925 50  0001 C CNN
+F 2 "KiCad/Resistors_SMD.pretty:R_0201" H 7900 2925 50  0001 C CNN
 F 3 "" H 7900 2925 50  0001 C CNN
 	1    7900 2925
@@
 F 0 "R202" H 2800 2425 59  0000 L BNN
 F 1 "10k" H 2800 2225 59  0000 L BNN
-F 2 "KiCad/Resistors_SMD.pretty:R_0402" H 2950 2375 50  0001 C CNN
+F 2 "KiCad/Resistors_SMD.pretty:R_0201" H 2950 2375 50  0001 C CNN
 F 3 "" H 2950 2375 50  0001 C CNN
 	1    2950 2375
@@
 F 0 "C206" H 3700 2725 59  0000 L BNN
 F 1 "1n" H 3900 2525 59  0000 L BNN
-F 2 "KiCad/Capacitors_SMD.pretty:C_0402" H 3800 2625 50  0001 C CNN
+F 2 "KiCad/Capacitors_SMD.pretty:C_0201" H 3800 2625 50  0001 C CNN
 F 3 "" H 3800 2625 50  0001 C CNN
 	1    3800 2625
@@
 F 0 "R206" H 4850 7325 59  0000 L BNN
 F 1 "750k" H 4850 7125 59  0000 L BNN
-F 2 "KiCad/Resistors_SMD.pretty:R_0402" H 5000 7275 50  0001 C CNN
+F 2 "KiCad/Resistors_SMD.pretty:R_0201" H 5000 7275 50  0001 C CNN
 F 3 "" H 5000 7275 50  0001 C CNN
 	1    5000 7275
@@
 F 0 "R207" H 4850 7925 59  0000 L BNN
 F 1 "240k" H 4850 7725 59  0000 L BNN
-F 2 "KiCad/Resistors_SMD.pretty:R_0402" H 5000 7875 50  0001 C CNN
+F 2 "KiCad/Resistors_SMD.pretty:R_0201" H 5000 7875 50  0001 C CNN
 F 3 "" H 5000 7875 50  0001 C CNN
 	1    5000 7875
@@
 F 0 "R204" H 4050 5725 59  0000 L BNN
 F 1 "1M" H 4050 5525 59  0000 L BNN
-F 2 "KiCad/Resistors_SMD.pretty:R_0402" H 4200 5675 50  0001 C CNN
+F 2 "KiCad/Resistors_SMD.pretty:R_0201" H 4200 5675 50  0001 C CNN
 F 3 "" H 4200 5675 50  0001 C CNN
 	1    4200 5675
@@
 F 0 "R209" H 5650 1675 59  0000 L BNN
 F 1 "330k" H 5650 1475 59  0000 L BNN
-F 2 "KiCad/Resistors_SMD.pretty:R_0402" H 5800 1625 50  0001 C CNN
+F 2 "KiCad/Resistors_SMD.pretty:R_0201" H 5800 1625 50  0001 C CNN
 F 3 "" H 5800 1625 50  0001 C CNN
 	1    5800 1625
@@
 F 0 "C202" V 1750 1150 59  0000 L BNN
 F 1 "100n" V 1525 1150 59  0000 L BNN
-F 2 "KiCad/Capacitors_SMD.pretty:C_0402" H 1575 1425 50  0001 C CNN
+F 2 "KiCad/Capacitors_SMD.pretty:C_0201" H 1575 1425 50  0001 C CNN
 F 3 "" H 1575 1425 50  0001 C CNN
 	1    1575 1425
@@
 F 0 "R205" H 4050 6625 59  0000 L BNN
 F 1 "10k" H 4050 6425 59  0000 L BNN
-F 2 "KiCad/Resistors_SMD.pretty:R_0402" H 4200 6575 50  0001 C CNN
+F 2 "KiCad/Resistors_SMD.pretty:R_0201" H 4200 6575 50  0001 C CNN
 F 3 "" H 4200 6575 50  0001 C CNN
 	1    4200 6575
@@
 F 0 "R211" H 6050 1675 59  0000 L BNN
 F 1 "10k" H 6050 1475 59  0000 L BNN
-F 2 "KiCad/Resistors_SMD.pretty:R_0402" H 6200 1625 50  0001 C CNN
+F 2 "KiCad/Resistors_SMD.pretty:R_0201" H 6200 1625 50  0001 C CNN
 F 3 "" H 6200 1625 50  0001 C CNN
 	1    6200 1625
@@
 F 0 "R208" H 5250 1075 59  0000 L BNN
 F 1 "47k" H 5250 875 59  0000 L BNN
-F 2 "KiCad/Resistors_SMD.pretty:R_0402" H 5400 1025 50  0001 C CNN
+F 2 "KiCad/Resistors_SMD.pretty:R_0201" H 5400 1025 50  0001 C CNN
 F 3 "" H 5400 1025 50  0001 C CNN
 	1    5400 1025
@@
 F 0 "R212" H 6250 7525 59  0000 L BNN
 F 1 "10k" H 6250 7325 59  0000 L BNN
-F 2 "KiCad/Resistors_SMD.pretty:R_0402" H 6400 7475 50  0001 C CNN
+F 2 "KiCad/Resistors_SMD.pretty:R_0201" H 6400 7475 50  0001 C CNN
 F 3 "" H 6400 7475 50  0001 C CNN
 	1    6400 7475
@@
 F 0 "R201" H 1750 7625 59  0000 L BNN
 F 1 "10k" H 1750 7425 59  0000 L BNN
-F 2 "KiCad/Resistors_SMD.pretty:R_0402" H 1900 7575 50  0001 C CNN
+F 2 "KiCad/Resistors_SMD.pretty:R_0201" H 1900 7575 50  0001 C CNN
 F 3 "" H 1900 7575 50  0001 C CNN
 	1    1900 7575
@@
 F 0 "C208" H 7625 1600 59  0000 L BNN
 F 1 "V 3p" H 8000 1575 59  0000 L BNN
-F 2 "KiCad/Capacitors_SMD.pretty:C_0402" H 7900 1725 50  0001 C CNN
+F 2 "KiCad/Capacitors_SMD.pretty:C_0201" H 7900 1725 50  0001 C CNN
 F 3 "" H 7900 1725 50  0001 C CNN
 	1    7900 1725
@@
 F 0 "C209" H 7650 1825 59  0000 L BNN
 F 1 "V 3p" H 8000 1800 59  0000 L BNN
-F 2 "KiCad/Capacitors_SMD.pretty:C_0402" H 7900 1925 50  0001 C CNN
+F 2 "KiCad/Capacitors_SMD.pretty:C_0201" H 7900 1925 50  0001 C CNN
 F 3 "" H 7900 1925 50  0001 C CNN
 	1    7900 1925
@@
 F 0 "C210" H 7650 2025 59  0000 L BNN
 F 1 "V 3p" H 8000 2025 59  0000 L BNN
-F 2 "KiCad/Capacitors_SMD.pretty:C_0402" H 7900 2125 50  0001 C CNN
+F 2 "KiCad/Capacitors_SMD.pretty:C_0201" H 7900 2125 50  0001 C CNN
 F 3 "" H 7900 2125 50  0001 C CNN
 	1    7900 2125
@@
 F 0 "C211" H 8000 2825 59  0000 L BNN
 F 1 "V 3p" H 8200 2625 59  0000 L BNN
-F 2 "KiCad/Capacitors_SMD.pretty:C_0402" H 8100 2725 50  0001 C CNN
+F 2 "KiCad/Capacitors_SMD.pretty:C_0201" H 8100 2725 50  0001 C CNN
 F 3 "" H 8100 2725 50  0001 C CNN
 	1    8100 2725
@@
 F 0 "C212" H 8300 2825 59  0000 L BNN
 F 1 "V 3p" H 8500 2625 59  0000 L BNN
-F 2 "KiCad/Capacitors_SMD.pretty:C_0402" H 8400 2725 50  0001 C CNN
+F 2 "KiCad/Capacitors_SMD.pretty:C_0201" H 8400 2725 50  0001 C CNN
 F 3 "" H 8400 2725 50  0001 C CNN
 	1    8400 2725
@@
 F 0 "C213" H 8600 2825 59  0000 L BNN
 F 1 "V 3p" H 8800 2625 59  0000 L BNN
-F 2 "KiCad/Capacitors_SMD.pretty:C_0402" H 8700 2725 50  0001 C CNN
+F 2 "KiCad/Capacitors_SMD.pretty:C_0201" H 8700 2725 50  0001 C CNN
 F 3 "" H 8700 2725 50  0001 C CNN
 	1    8700 2725
@@
 F 0 "R203" H 3650 7925 59  0000 L BNN
 F 1 "10k" H 3650 7725 59  0000 L BNN
-F 2 "KiCad/Resistors_SMD.pretty:R_0402" H 3800 7875 50  0001 C CNN
+F 2 "KiCad/Resistors_SMD.pretty:R_0201" H 3800 7875 50  0001 C CNN
 F 3 "" H 3800 7875 50  0001 C CNN
 	1    3800 7875
@@
 F 0 "R213" H 6550 7025 59  0000 L BNN
 F 1 "10k" H 6550 6825 59  0000 L BNN
-F 2 "KiCad/Resistors_SMD.pretty:R_0402" H 6700 6975 50  0001 C CNN
+F 2 "KiCad/Resistors_SMD.pretty:R_0201" H 6700 6975 50  0001 C CNN
 F 3 "" H 6700 6975 50  0001 C CNN
 	1    6700 6975
@@
 F 0 "R210" H 5750 7525 59  0000 L BNN
 F 1 "10k" H 5750 7325 59  0000 L BNN
-F 2 "KiCad/Resistors_SMD.pretty:R_0402" H 5900 7475 50  0001 C CNN
+F 2 "KiCad/Resistors_SMD.pretty:R_0201" H 5900 7475 50  0001 C CNN
 F 3 "" H 5900 7475 50  0001 C CNN
 	1    5900 7475

Commit message: Make ISP header a pogo pin one
Parts:
- X202: footprint component_tester:WANNE6_PCBKANTE -> component_tester:Pin_Header_Straight_2x03_Pitch1.27mm
Changed lines of the file:
@@
 F 0 "X202" H 8450 4775 42  0000 L BNN
 F 1 "ISP" H 8450 4425 42  0000 L BNN
-F 2 "component_tester:WANNE6_PCBKANTE" H 8500 4625 50  0001 C CNN
+F 2 "component_tester:Pin_Header_Straight_2x03_Pitch1.27mm" H 8500 4625 50  0001 C CNN
 F 3 "" H 8500 4625 50  0001 C CNN
 	1    8500 4625

Commit message: Cut out precision voltage reference
Parts:
- removed D202: LM4040A-2V5, component_tester:SOT23, symbol component_tester-eagle-import:LM4040
- removed R208: 47k, KiCad/Resistors_SMD.pretty:R_0201, symbol component_tester-eagle-import:R0805
- C202: footprint KiCad/Capacitors_SMD.pretty:C_0201 -> KiCad/Capacitors_SMD.pretty:C_0402
Connections:
- wire segments 213 -> 206
Changed lines of the file:
@@
 	5800 1425 5800 825
-Wire Wire Line
-	5400 1825 5400 1925
 Wire Wire Line
 	1700 6475 1700 7275
@@
 	2250 2375 2750 2375
 Wire Wire Line
-	5400 725  5400 825
-Wire Wire Line
 	6200 725  6200 1425
 Wire Wire Line
@@
 	5700 6575 5700 8375
 Connection ~ 5700 6575
-Wire Wire Line
-	5400 1225 5400 1325
-Wire Wire Line
-	5400 1325 5400 1425
-Wire Wire Line
-	5600 1325 5400 1325
-Connection ~ 5400 1325
 Wire Wire Line
 	3300 5675 4000 5675
@@
 F 0 "C202" V 1750 1150 59  0000 L BNN
 F 1 "100n" V 1525 1150 59  0000 L BNN
-F 2 "KiCad/Capacitors_SMD.pretty:C_0201" H 1575 1425 50  0001 C CNN
+F 2 "KiCad/Capacitors_SMD.pretty:C_0402" H 1575 1425 50  0001 C CNN
 F 3 "" H 1575 1425 50  0001 C CNN
 	1    1575 1425
@@
 	1    6200 1625
 	0    -1   -1   0
-$EndComp
-$Comp
-L component_tester-eagle-import:LM4040 D202
-U 1 0 D58447641462D966
-P 5400 1625
-F 0 "D202" H 5500 1725 59  0000 L BNN
-F 1 "LM4040A-2V5" H 5500 1525 59  0000 L BNN
-F 2 "component_tester:SOT23" H 5400 1625 50  0001 C CNN
-F 3 "" H 5400 1625 50  0001 C CNN
-	1    5400 1625
-	0    -1   -1   0
-$EndComp
-$Comp
-L component_tester-eagle-import:R0805 R208
-U 1 0 E4B58C2114CE6AAC
-P 5400 1025
-F 0 "R208" H 5250 1075 59  0000 L BNN
-F 1 "47k" H 5250 875 59  0000 L BNN
-F 2 "KiCad/Resistors_SMD.pretty:R_0201" H 5400 1025 50  0001 C CNN
-F 3 "" H 5400 1025 50  0001 C CNN
-	1    5400 1025
-	0    -1   -1   0
-$EndComp
-$Comp
-L component_tester-eagle-import:+5V #+5V0204
-U 1 0 534DB015CAF7019A
-P 5400 625
-F 0 "#+5V0204" H 5400 625 50  0001 C CNN
-F 1 "+5V" V 5300 425 59  0000 L BNN
-F 2 "" H 5400 625 50  0001 C CNN
-F 3 "" H 5400 625 50  0001 C CNN
-	1    5400 625
-	1    0    0    -1
-$EndComp
-$Comp
-L component_tester-eagle-import:GND #GND0211
-U 1 0 E847186D109F320A
-P 5400 2025
-F 0 "#GND0211" H 5400 2025 50  0001 C CNN
-F 1 "GND" H 5300 1925 59  0000 L BNN
-F 2 "" H 5400 2025 50  0001 C CNN
-F 3 "" H 5400 2025 50  0001 C CNN
-	1    5400 2025
-	1    0    0    -1
 $EndComp
 $Comp
@@
 	5600 2925 5600 5675
 Wire Wire Line
-	5600 2825 5400 2825
-Wire Wire Line
-	5600 1325 5600 2825
-Wire Wire Line
 	5400 2725 6600 2725

Commit message: Switch some transistors for smaller footprints
Parts:
- D201: footprint component_tester:SOT23 -> digikey/digikey-kicad-library/src/Source_Footprints:SOT-523; MPN1 (none) -> BAV99T-7-F; MPN2 (none) -> BAV99T
- D203: footprint component_tester:SOT23 -> KiCad/LEDs.pretty:LED_0402; MPN (none) -> BAS40LP-7
- T203: footprint component_tester:SOT23 -> KiCad/TO_SOT_Packages_SMD.pretty:SOT-323_SC-70; MPN (none) -> BSS123W-7-F
- T204: footprint component_tester:SOT23 -> digikey/digikey-kicad-library/src/Source_Footprints:SOT-523; MPN (none) -> BC847AT-7-F
Other:
- note added: "+BATT = 3V von Lithiumzelle"
- note removed: "BAT+ = 3V von Lithiumzelle"
Changed lines of the file:
@@
 U 1 0 7513E83E99E27C05
 P 2900 7375
-F 0 "C203" V 2850 7525 59  0000 L BNN
+F 0 "C203" V 2875 7425 59  0000 L BNN
 F 1 "47u" V 3075 7500 59  0000 L BNN
 F 2 "KiCad/Capacitors_SMD.pretty:C_0805" H 2900 7375 50  0001 C CNN
@@
 F 0 "T204" H 7100 7025 59  0000 L BNN
 F 1 "BC847" H 7100 6925 59  0000 L BNN
-F 2 "component_tester:SOT23" H 7000 6975 50  0001 C CNN
+F 2 "digikey/digikey-kicad-library/src/Source_Footprints:SOT-523" H 7000 6975 50  0001 C CNN
 F 3 "" H 7000 6975 50  0001 C CNN
+F 4 "BC847AT-7-F" H 7000 6975 50  0001 C CNN "MPN"
 	1    7000 6975
 	1    0    0    -1
@@
 F 0 "D201" H 2400 6875 59  0000 L BNN
 F 1 "BAV99" H 2450 6425 59  0000 L BNN
-F 2 "component_tester:SOT23" H 2500 6675 50  0001 C CNN
+F 2 "digikey/digikey-kicad-library/src/Source_Footprints:SOT-523" H 2500 6675 50  0001 C CNN
 F 3 "" H 2500 6675 50  0001 C CNN
+F 4 "BAV99T-7-F" H 2500 6675 50  0001 C CNN "MPN1"
+F 5 "BAV99T" H 2500 6675 50  0001 C CNN "MPN2"
 	1    2500 6675
 	0    1    1    0
@@
 F 0 "D203" H 6200 7075 59  0000 L BNN
 F 1 "BAS40" H 6200 6875 59  0000 L BNN
-F 2 "component_tester:SOT23" H 6100 6975 50  0001 C CNN
+F 2 "KiCad/LEDs.pretty:LED_0402" H 6100 6975 50  0001 C CNN
 F 3 "" H 6100 6975 50  0001 C CNN
+F 4 "BAS40LP-7" H 6100 6975 50  0001 C CNN "MPN"
 	1    6100 6975
 	1    0    0    -1
@@
 VI = Spannungsregler-Eingang
 Text Notes 9200 6000 0    85   ~ 0
-BAT+ = 3V von Lithiumzelle
++BATT = 3V von Lithiumzelle
 Text Notes 725  725  0    127  ~ 0
 K.-H. Kübbeler, DF3DCB, DH8GHH
@@
 F 0 "T203" H 6300 5550 59  0000 L BNN
 F 1 "BSS123" H 6300 5450 59  0000 L BNN
-F 2 "component_tester:SOT23" H 6200 5550 50  0001 C CNN
+F 2 "KiCad/TO_SOT_Packages_SMD.pretty:SOT-323_SC-70" H 6200 5550 50  0001 C CNN
 F 3 "" H 6200 5550 50  0001 C CNN
+F 4 "BSS123W-7-F" H 6200 5550 50  0001 C CNN "MPN"
 	1    6200 5550
 	1    0    0    -1
