File: kicad/component_tester_2.sch (KiCad schematic (older format))
At the start: 12 parts, among them IC3 MAX1811, IC4 FT232RL, J1 0R-JUMPA, J2 0R-JUMPA, T4 BSS123, X13 STIFT, X14 STIFT

Commit message: Delete eagle schematic blocks
Other:
- note removed: ">REV"
- note removed: "Optionen"
Changed lines of the file:
@@
 $Descr User 12098 8268
 encoding utf-8
-Sheet 1 3
+Sheet 3 3
 Title ""
 Date ""
@@
 $EndComp
 $Comp
-L component_tester-eagle-import:DINA4_L #FRAME2
-U 2 0 D06FCA34DFE0E5AC
-P 7300 6700
-AR Path="/D06FCA34DFE0E5AC" Ref="#FRAME2"  Part="2"
-AR Path="/5B1C713A/D06FCA34DFE0E5AC" Ref="#FRAME2"  Part="2"
-F 0 "#FRAME2" H 7300 6700 50  0001 C CNN
-F 1 "DINA4_L" H 7300 6700 50  0001 C CNN
-F 2 "" H 7300 6700 50  0001 C CNN
-F 3 "" H 7300 6700 50  0001 C CNN
-	2    7300 6700
-	1    0    0    -1
-$EndComp
-$Comp
 L component_tester-eagle-import:GND #GND24
 U 1 0 D2BA7EC8664B2FAE
@@
 	-1   0    0    1
 $EndComp
-Text Notes 7500 5700 0    254  ~ 0
-Optionen
-Text Notes 10900 6400 0    100  ~ 0
->REV
 Text Notes 1600 1700 0    170  ~ 0
 Option USB-Ausgabe

Commit message: Switch resistors and caps to 0201 where possible
Parts:
- C13: footprint component_tester:C0805 -> KiCad/Capacitors_SMD.pretty:C_0805
- R22: footprint component_tester:R0805 -> KiCad/Resistors_SMD.pretty:R_0201
Changed lines of the file:
@@
 F 0 "C13" H 5300 4400 59  0000 L BNN
 F 1 "100n" H 5500 4200 59  0000 L BNN
-F 2 "component_tester:C0805" H 5400 4300 50  0001 C CNN
+F 2 "KiCad/Capacitors_SMD.pretty:C_0805" H 5400 4300 50  0001 C CNN
 F 3 "" H 5400 4300 50  0001 C CNN
 	1    5400 4300
@@
 F 0 "R22" H 10050 2350 59  0000 L BNN
 F 1 "100" H 10050 2150 59  0000 L BNN
-F 2 "component_tester:R0805" H 10200 2300 50  0001 C CNN
+F 2 "KiCad/Resistors_SMD.pretty:R_0201" H 10200 2300 50  0001 C CNN
 F 3 "" H 10200 2300 50  0001 C CNN
 	1    10200 2300

Commit message: Sort out ground net
Changed lines of the file:
@@
 Wire Wire Line
 	8600 3700 8600 3500
-Text GLabel 8600 3700 0    10   BiDi ~ 0
-GND
 Wire Wire Line
 	8800 3700 8800 3500
-Text GLabel 8800 3700 0    10   BiDi ~ 0
-GND
 Wire Wire Line
 	8300 3000 7900 3000
@@
 Wire Wire Line
 	10500 3700 10500 3300
-Text GLabel 10500 3700 0    10   BiDi ~ 0
-GND
 Wire Wire Line
 	9600 3600 9600 3700
-Text GLabel 9600 3600 0    10   BiDi ~ 0
-GND
 Wire Wire Line
 	9900 3600 9900 3700
-Text GLabel 9900 3600 0    10   BiDi ~ 0
-GND
 Wire Wire Line
 	7900 2100 7900 2300
@@
 VCC
 Wire Wire Line
-	9600 3300 9600 3000
-Wire Wire Line
 	9600 3000 9100 3000
 Wire Wire Line
@@
 	9600 3000 9600 2000
 Connection ~ 9600 3000
-Text GLabel 9600 3300 0    10   BiDi ~ 0
-BAT+
 Wire Wire Line
 	7700 2800 8300 2800
@@
 $EndComp
 $Comp
-L component_tester-eagle-import:+5V #+5V10
-U 1 0 6DC7F6CC0F3D497E
-P 9600 1900
-AR Path="/6DC7F6CC0F3D497E" Ref="#+5V10"  Part="1"
-AR Path="/5B1C713A/6DC7F6CC0F3D497E" Ref="#+5V010"  Part="1"
-F 0 "#+5V010" H 9600 1900 50  0001 C CNN
-F 1 "BAT+" V 9500 1700 59  0000 L BNN
-F 2 "" H 9600 1900 50  0001 C CNN
-F 3 "" H 9600 1900 50  0001 C CNN
-	1    9600 1900
-	1    0    0    -1
-$EndComp
-$Comp
 L component_tester-eagle-import:STIFT X14
 U 1 0 BD362AB30D38F6C5
@@
 Text Notes 7100 1700 0    170  ~ 0
 Option Li+ Charger
+Text GLabel 8600 3700 0    10   BiDi ~ 0
+GND
+Text GLabel 8800 3700 0    10   BiDi ~ 0
+GND
+Text GLabel 10500 3700 0    10   BiDi ~ 0
+GND
+Text GLabel 9900 3600 0    10   BiDi ~ 0
+GND
+Text GLabel 9600 3600 0    10   BiDi ~ 0
+GND
+Wire Wire Line
+	9600 3300 9600 3000
+$Comp
+L component_tester-eagle-import:+5V #+5V10
+U 1 0 6DC7F6CC0F3D497E
+P 9600 1900
+AR Path="/6DC7F6CC0F3D497E" Ref="#+5V10"  Part="1"
+AR Path="/5B1C713A/6DC7F6CC0F3D497E" Ref="#+5V010"  Part="1"
+F 0 "#+5V010" H 9600 1900 50  0001 C CNN
+F 1 "BAT+" V 9500 1700 59  0000 L BNN
+F 2 "" H 9600 1900 50  0001 C CNN
+F 3 "" H 9600 1900 50  0001 C CNN
+	1    9600 1900
+	1    0    0    -1
+$EndComp
 $EndSCHEMATC

Commit message: Sort out power nets/labels
Parts:
- removed X13, X14: STIFT, component_tester:STIFT, symbol component_tester-eagle-import:STIFT
Connections:
- net labels added: +BATT
- net labels removed: BAT+
- wire segments 49 -> 47
Changed lines of the file:
@@
 Connection ~ 3700 2200
 Connection ~ 3700 2300
-Text GLabel 3900 2200 0    10   BiDi ~ 0
-GND
 Wire Wire Line
 	5000 2400 5400 2400
-Text GLabel 5000 2400 0    10   BiDi ~ 0
-GND
 Wire Wire Line
 	5400 4400 5400 4600
-Text GLabel 5400 4400 0    10   BiDi ~ 0
-GND
 Wire Wire Line
 	8600 3700 8600 3500
@@
 Wire Wire Line
 	7900 3000 7900 3700
-Text GLabel 8300 3000 0    10   BiDi ~ 0
-GND
 Wire Wire Line
 	7600 2900 7600 3700
-Text GLabel 7600 2900 0    10   BiDi ~ 0
-GND
-Wire Wire Line
-	10500 3700 10500 3300
 Wire Wire Line
 	9600 3600 9600 3700
@@
 Wire Wire Line
 	7900 2300 8100 2300
-Text GLabel 7900 2100 0    10   BiDi ~ 0
-GND
 Wire Wire Line
 	3000 3900 2400 3900
@@
 Wire Wire Line
 	7600 2700 7600 2100
-Text GLabel 7600 2700 0    10   BiDi ~ 0
-VCC
 Wire Wire Line
 	9900 2800 9900 3300
@@
 Connection ~ 9900 2800
 Connection ~ 9300 2800
-Text GLabel 9900 2800 0    10   BiDi ~ 0
-VCC
 Wire Wire Line
 	10200 2000 10200 2100
-Text GLabel 10200 2000 0    10   BiDi ~ 0
-VCC
 Wire Wire Line
 	3300 4500 3300 4100
-Text GLabel 3300 4500 0    10   BiDi ~ 0
-VCC
 Wire Wire Line
 	9600 3000 9100 3000
-Wire Wire Line
-	9600 3000 10500 3000
-Wire Wire Line
-	9600 3000 9600 2000
-Connection ~ 9600 3000
 Wire Wire Line
 	7700 2800 8300 2800
@@
 $EndComp
 $Comp
-L component_tester-eagle-import:STIFT X13
-U 1 0 9F58853A4C8084F3
-P 10500 3000
-AR Path="/9F58853A4C8084F3" Ref="X13"  Part="1"
-AR Path="/5B1C713A/9F58853A4C8084F3" Ref="X13"  Part="1"
-F 0 "X13" H 10450 3050 42  0000 L BNN
-F 1 "STIFT" H 10450 2900 42  0000 L BNN
-F 2 "component_tester:STIFT" H 10500 3000 50  0001 C CNN
-F 3 "" H 10500 3000 50  0001 C CNN
-	1    10500 3000
-	1    0    0    -1
-$EndComp
-$Comp
 L component_tester-eagle-import:R0805 R22
 U 1 0 8CA68C2673741284
@@
 F 3 "" H 10200 1900 50  0001 C CNN
 	1    10200 1900
-	1    0    0    -1
-$EndComp
-$Comp
-L component_tester-eagle-import:STIFT X14
-U 1 0 BD362AB30D38F6C5
-P 10500 3300
-AR Path="/BD362AB30D38F6C5" Ref="X14"  Part="1"
-AR Path="/5B1C713A/BD362AB30D38F6C5" Ref="X14"  Part="1"
-F 0 "X14" H 10450 3350 42  0000 L BNN
-F 1 "STIFT" H 10450 3200 42  0000 L BNN
-F 2 "component_tester:STIFT" H 10500 3300 50  0001 C CNN
-F 3 "" H 10500 3300 50  0001 C CNN
-	1    10500 3300
-	1    0    0    -1
-$EndComp
-$Comp
-L component_tester-eagle-import:GND #GND36
-U 1 0 61F5680C397F6EFB
-P 10500 3800
-AR Path="/61F5680C397F6EFB" Ref="#GND36"  Part="1"
-AR Path="/5B1C713A/61F5680C397F6EFB" Ref="#GND036"  Part="1"
-F 0 "#GND036" H 10500 3800 50  0001 C CNN
-F 1 "GND" H 10400 3700 59  0000 L BNN
-F 2 "" H 10500 3800 50  0001 C CNN
-F 3 "" H 10500 3800 50  0001 C CNN
-	1    10500 3800
 	1    0    0    -1
 $EndComp
@@
 Text Notes 7100 1700 0    170  ~ 0
 Option Li+ Charger
-Text GLabel 8600 3700 0    10   BiDi ~ 0
-GND
-Text GLabel 8800 3700 0    10   BiDi ~ 0
-GND
-Text GLabel 10500 3700 0    10   BiDi ~ 0
-GND
-Text GLabel 9900 3600 0    10   BiDi ~ 0
-GND
-Text GLabel 9600 3600 0    10   BiDi ~ 0
-GND
 Wire Wire Line
 	9600 3300 9600 3000
-$Comp
-L component_tester-eagle-import:+5V #+5V10
-U 1 0 6DC7F6CC0F3D497E
-P 9600 1900
-AR Path="/6DC7F6CC0F3D497E" Ref="#+5V10"  Part="1"
-AR Path="/5B1C713A/6DC7F6CC0F3D497E" Ref="#+5V010"  Part="1"
-F 0 "#+5V010" H 9600 1900 50  0001 C CNN
-F 1 "BAT+" V 9500 1700 59  0000 L BNN
-F 2 "" H 9600 1900 50  0001 C CNN
-F 3 "" H 9600 1900 50  0001 C CNN
-	1    9600 1900
-	1    0    0    -1
-$EndComp
+Wire Wire Line
+	9600 3000 9600 2000
+Connection ~ 9600 3000
+$Comp
+L power:+BATT #PWR?
+U 1 1 5B67D634
+P 9600 2000
+F 0 "#PWR?" H 9600 1850 50  0001 C CNN
+F 1 "+BATT" H 9615 2173 50  0000 C CNN
+F 2 "" H 9600 2000 50  0001 C CNN
+F 3 "" H 9600 2000 50  0001 C CNN
+	1    9600 2000
+	1    0    0    -1
+$EndComp

Commit message: Import Adafruit OLED breakout
Parts:
- renumbered C13 to C301, C16 to C302, C17 to C303, IC4 to IC301, IC3 to IC302, J1 to J301, J2 to J302, LED1 to LED301, R22 to R301, T4 to T301

Commit message: Switch 0201 footprints for 0402
Parts:
- R301: footprint KiCad/Resistors_SMD.pretty:R_0201 -> KiCad/Resistors_SMD.pretty:R_0402
Changed lines of the file:
@@
 F 0 "R301" H 10050 2350 59  0000 L BNN
 F 1 "100" H 10050 2150 59  0000 L BNN
-F 2 "KiCad/Resistors_SMD.pretty:R_0201" H 10200 2300 50  0001 C CNN
+F 2 "KiCad/Resistors_SMD.pretty:R_0402" H 10200 2300 50  0001 C CNN
 F 3 "" H 10200 2300 50  0001 C CNN
 	1    10200 2300
