File: kicad/component_tester_3.sch (KiCad schematic (older format))
At the start: 26 parts, among them Q401 BSS138, Q402 BSS138, U401 VREG_SOT23-5

Commit message: Remove unnecessary stuff from OLED circuitry
Parts:
- removed C401, C402: 10uF, KiCad/Capacitors_SMD.pretty:C_0805, symbol Adafruit_128x64_Mono_OLED_PCB_v2-eagle-import:CAP_CERAMIC0805
- removed SJ401, SJ402: SOLDERJUMPERREFLOW_NOPASTE, Adafruit 128x64 Mono OLED PCB v2:SOLDERJUMPER_REFLOW_NOPASTE, symbol Adafruit_128x64_Mono_OLED_PCB_v2-eagle-import:SOLDERJUMPERREFLOW_NOPASTE
- removed U401: VREG_SOT23-5, Adafruit 128x64 Mono OLED PCB v2:SOT23-5, symbol Adafruit_128x64_Mono_OLED_PCB_v2-eagle-import:VREG_SOT23-5
Connections:
- net labels added: +5V, +BATT
- net labels removed: VIN
- wire segments 118 -> 93
Other:
- note removed: "Bus default = SPI4"
- note removed: "Close SJ2 for I2C"
- note removed: "Close for"
- note removed: "I2C"
- note removed: "ToDo: Change address to default low"

Commit message: Switch back to 0201s and continue placing
Parts:
- R401, R402, R403, R404, R405, R406, R407, R408, R409: footprint KiCad/Resistors_SMD.pretty:R_0402 -> KiCad/Resistors_SMD.pretty:R_0201
Changed lines of the file:
@@
 F 0 "R408" H 7300 4080 50  0000 L BNN
 F 1 "10K" H 7300 3875 50  0000 L BNN
-F 2 "KiCad/Resistors_SMD.pretty:R_0402" H 7400 4000 50  0001 C CNN
+F 2 "KiCad/Resistors_SMD.pretty:R_0201" H 7400 4000 50  0001 C CNN
 F 3 "" H 7400 4000 50  0001 C CNN
 	1    7400 4000
@@
 F 0 "R405" H 6600 1380 50  0000 L BNN
 F 1 "10K" H 6600 1175 50  0000 L BNN
-F 2 "KiCad/Resistors_SMD.pretty:R_0402" H 6700 1300 50  0001 C CNN
+F 2 "KiCad/Resistors_SMD.pretty:R_0201" H 6700 1300 50  0001 C CNN
 F 3 "" H 6700 1300 50  0001 C CNN
 	1    6700 1300
@@
 F 0 "R406" H 6900 1380 50  0000 L BNN
 F 1 "10K" H 6900 1175 50  0000 L BNN
-F 2 "KiCad/Resistors_SMD.pretty:R_0402" H 7000 1300 50  0001 C CNN
+F 2 "KiCad/Resistors_SMD.pretty:R_0201" H 7000 1300 50  0001 C CNN
 F 3 "" H 7000 1300 50  0001 C CNN
 	1    7000 1300
@@
 F 0 "R407" H 7200 1380 50  0000 L BNN
 F 1 "10K" H 7200 1175 50  0000 L BNN
-F 2 "KiCad/Resistors_SMD.pretty:R_0402" H 7300 1300 50  0001 C CNN
+F 2 "KiCad/Resistors_SMD.pretty:R_0201" H 7300 1300 50  0001 C CNN
 F 3 "" H 7300 1300 50  0001 C CNN
 	1    7300 1300
@@
 F 0 "R401" H 2500 3180 50  0000 L BNN
 F 1 "10K" H 2500 2975 50  0000 L BNN
-F 2 "KiCad/Resistors_SMD.pretty:R_0402" H 2600 3100 50  0001 C CNN
+F 2 "KiCad/Resistors_SMD.pretty:R_0201" H 2600 3100 50  0001 C CNN
 F 3 "" H 2600 3100 50  0001 C CNN
 	1    2600 3100
@@
 F 0 "R402" H 2800 3180 50  0000 L BNN
 F 1 "10K" H 2800 2975 50  0000 L BNN
-F 2 "KiCad/Resistors_SMD.pretty:R_0402" H 2900 3100 50  0001 C CNN
+F 2 "KiCad/Resistors_SMD.pretty:R_0201" H 2900 3100 50  0001 C CNN
 F 3 "" H 2900 3100 50  0001 C CNN
 	1    2900 3100
@@
 F 0 "R403" H 3700 3180 50  0000 L BNN
 F 1 "10K" H 3700 2975 50  0000 L BNN
-F 2 "KiCad/Resistors_SMD.pretty:R_0402" H 3800 3100 50  0001 C CNN
+F 2 "KiCad/Resistors_SMD.pretty:R_0201" H 3800 3100 50  0001 C CNN
 F 3 "" H 3800 3100 50  0001 C CNN
 	1    3800 3100
@@
 F 0 "R404" H 4000 3180 50  0000 L BNN
 F 1 "10K" H 4000 2975 50  0000 L BNN
-F 2 "KiCad/Resistors_SMD.pretty:R_0402" H 4100 3100 50  0001 C CNN
+F 2 "KiCad/Resistors_SMD.pretty:R_0201" H 4100 3100 50  0001 C CNN
 F 3 "" H 4100 3100 50  0001 C CNN
 	1    4100 3100
@@
 F 0 "R409" H 8600 5180 50  0000 L BNN
 F 1 "390K" H 8600 4975 50  0000 L BNN
-F 2 "KiCad/Resistors_SMD.pretty:R_0402" H 8700 5100 50  0001 C CNN
+F 2 "KiCad/Resistors_SMD.pretty:R_0201" H 8700 5100 50  0001 C CNN
 F 3 "" H 8700 5100 50  0001 C CNN
 	1    8700 5100
