File: kicad/component_tester.kicad_pcb (KiCad board)
At the start: 4 copper layers, 100.4 x 83 mm, 81 parts, among them IC201 MCP1640, IC202 ATmega328P-MMH, IC301 FT232RL, IC302 MAX1811, J301 0R-JUMPA, J302 0R-JUMPA, Q201 8 MHz, Q401 BSS138, Q402 BSS138, SW201 EVQ, T201 PMV65XP, T202 BSS84, T203 BSS123, T204 BC847, T301 BSS123, X201 MICRO-USB, X202 ISP

Commit message: Do some routing
Parts:
- moved C203 95.2 mm to (194.8, 113.5)
- moved D203 84.1 mm to (201.5, 113.5), turned to 270 degrees
- moved T204 80.7 mm to (199.4, 97.4)
- moved C206 68.7 mm to (168.2, 109.4)
- moved L201 38.8 mm to (201.4, 108.6)
- moved IC201 34.7 mm to (196.1, 109.0)
- moved T202 30.2 mm to (196.3, 104.8)
- moved C202 1.08 mm to (169.7, 109.2)
- moved C201 0.91 mm to (168.6, 110.9)
- moved IC202 0.91 mm to (173.0, 109.2)
- moved R217 0.15 mm to (177.6, 110.1)
- moved R214 0.14 mm to (179.0, 111.4)
- moved R215 0.14 mm to (177.7, 111.4)
- moved C210 0.06 mm to (180.6, 111.3), turned to 0 degrees
- moved C212 0.05 mm to (179.0, 110.2), turned to 180 degrees
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Routing:
- net Net-(C208-Pad1): track 0.00 -> 29.2 mm, vias 0 -> 2
- net Net-(IC202-Pad15): track 0.00 -> 18.9 mm
- net Net-(C210-Pad1): track 0.00 -> 18.7 mm
- net Net-(IC202-Pad14): track 0.00 -> 16.6 mm, vias 0 -> 2
- net GND: track 2.81 -> 16.8 mm, vias 2 -> 5
- net +5V: track 2.80 -> 11.3 mm, vias 0 -> 2
- net Net-(IC202-Pad13): track 0.00 -> 8.20 mm, vias 0 -> 2
- net Net-(IC202-Pad12): track 0.00 -> 7.56 mm, vias 0 -> 2
- net Net-(IC202-Pad10): track 0.00 -> 6.71 mm
- net Net-(IC202-Pad11): track 0.00 -> 6.31 mm
- net Net-(C209-Pad1): track 0.00 -> 4.05 mm
- net Net-(C206-Pad2): track 0.00 -> 2.13 mm
